Commit message: trying to update cad, but failing to run meldis

File: models/wing_asy/urdf/wing_asy.urdf (robot description, URDF)
Before this commit: robot wing_asy, 3 links, 2 joints
Links:
- link part_1: geometry visual mesh filename=package://wing_asy/meshes/Part_1.obj scale=1 1 1
- link part_1_1: geometry visual mesh filename=package://wing_asy/meshes/Part_1_1.obj scale=1 1 1
Joints:
- removed joint hanging_node_to_root_joint
- added joint fastened_2: type fixed, parent root, child part_1, origin xyz=0 0 1.35525e-20 rpy=0 -0 0, axis 0 0 1
- joint fastened_1: child part_1 -> part_1_1; origin xyz=-0.00679779 0.00217114 1.5e-06 rpy=0 -0 0 -> xyz=0 0 -8e-05 rpy=0 -0 0; parent part_1_1 -> part_1

File: models/wing_asy/urdf/wing_asy_visualizer.urdf (robot description, URDF)
Before this commit: robot wing_asy_visualizer, 3 links, 2 joints
Links:
- link part_1: mass None -> 3.83835e-10; geometry visual mesh filename=../meshes/Part_1.obj scale=1 1 1
- link part_1_1: mass None -> 8.16534e-11; geometry visual mesh filename=../meshes/Part_1_1.obj scale=1 1 1
Joints:
- removed joint hanging_node_to_root_joint
- added joint fastened_2: type fixed, parent root, child part_1, origin xyz=0 0 1.35525e-20 rpy=0 -0 0, axis 0 0 1
- joint fastened_1: axis (none) -> 0 0 -1; child part_1 -> part_1_1; origin xyz=-0.679779 0.217114 0.00015 rpy=0 -0 0 -> xyz=0 0 -8e-05 rpy=0 -0 0; parent part_1_1 -> part_1

File: models/wing_asy_right/urdf/wing_asy_right.urdf (robot description, URDF)
Before this commit: robot wing_asy_right, 3 links, 2 joints
Links:
- link part_1: geometry visual mesh filename=package://wing_asy_right/meshes/Part_1.obj scale=1 1 1
- link part_1_1: geometry visual mesh filename=package://wing_asy_right/meshes/Part_1_1.obj scale=1 1 1
Joints:
- removed joint hanging_node_to_root_joint
- added joint group_1_fastened_joint: type fixed, parent part_1_1, child part_1, origin xyz=0.00679779 -0.00217114 8e-05 rpy=0 0 -2.76357e-75, axis 0 0 1
- joint fastened_1: child part_1 -> part_1_1; origin xyz=-0.00661946 0.00191632 8e-05 rpy=1.6673e-92 1.75162e-46 1.90372e-46 -> xyz=1.21431e-17 -2.81893e-18 -1.142e-33 rpy=-3.14159 -2.18953e-46 3.14159; parent part_1_1 -> root

File: models/wing_asy_right/urdf/wing_asy_right_visualizer.urdf (robot description, URDF)
Before this commit: robot wing_asy_right_visualizer, 3 links, 2 joints
Links:
- link part_1: geometry visual mesh filename=../meshes/Part_1.obj scale=1 1 1
- link part_1_1: geometry visual mesh filename=../meshes/Part_1_1.obj scale=1 1 1
Joints:
- removed joint hanging_node_to_root_joint
- added joint group_1_fastened_joint: type fixed, parent part_1_1, child part_1, origin xyz=0.00679779 -0.00217114 8e-05 rpy=0 0 -2.76357e-75, axis 0 0 1
- joint fastened_1: child part_1 -> part_1_1; origin xyz=-0.661946 0.191632 0.008 rpy=1.6673e-92 1.75162e-46 1.90372e-46 -> xyz=1.21431e-17 -2.81893e-18 -1.142e-33 rpy=-3.14159 -2.18953e-46 3.14159; parent part_1_1 -> root

Commit message: revert

File: models/wing_asy/urdf/wing_asy.urdf (robot description, URDF)
Before this commit: robot wing_asy, 3 links, 2 joints
Links:
- link part_1: geometry visual mesh filename=package://wing_asy/meshes/Part_1.stl scale=1 1 1
- link part_1_1: geometry visual mesh filename=package://wing_asy/meshes/Part_1_1.stl scale=1 1 1
Joints:
- removed joint fastened_2
- added joint hanging_node_to_root_joint: type fixed, parent root, child part_1_1, origin xyz=0.000383789 -0.00139453 0.000726211 rpy=0 -0 0, axis 0 0 1
- joint fastened_1: child part_1_1 -> part_1; origin xyz=0 0 -8e-05 rpy=0 -0 0 -> xyz=-0.00679779 0.00217114 1.5e-06 rpy=0 -0 0; parent part_1 -> part_1_1

File: models/wing_asy/urdf/wing_asy_visualizer.urdf (robot description, URDF)
Before this commit: robot wing_asy_visualizer, 3 links, 2 joints
Links:
- link part_1: mass 3.83835e-10 -> None; geometry visual mesh filename=../meshes/Part_1.stl scale=100 100 100
- link part_1_1: mass 8.16534e-11 -> None; geometry visual mesh filename=../meshes/Part_1_1.stl scale=100 100 100
Joints:
- removed joint fastened_2
- added joint hanging_node_to_root_joint: type fixed, parent root, child part_1_1, origin xyz=0.0383789 -0.139453 0.0726211 rpy=0 -0 0
- joint fastened_1: axis 0 0 -1 -> (none); child part_1_1 -> part_1; origin xyz=0 0 -8e-05 rpy=0 -0 0 -> xyz=-0.679779 0.217114 0.00015 rpy=0 -0 0; parent part_1 -> part_1_1

File: models/wing_asy_right/urdf/wing_asy_right.urdf (robot description, URDF)
Before this commit: robot wing_asy_right, 3 links, 2 joints
Links:
- link part_1: geometry visual mesh filename=package://wing_asy_right/meshes/Part_1.stl scale=1 1 1
- link part_1_1: geometry visual mesh filename=package://wing_asy_right/meshes/Part_1_1.stl scale=1 1 1
Joints:
- removed joint group_1_fastened_joint
- added joint hanging_node_to_root_joint: type fixed, parent root, child part_1_1, origin xyz=0.00186505 0.00121117 0.000640399 rpy=-3.14159 1.99562e-30 -3.14159, axis 0 0 1
- joint fastened_1: child part_1_1 -> part_1; origin xyz=1.21431e-17 -2.81893e-18 -1.142e-33 rpy=-3.14159 -2.18953e-46 3.14159 -> xyz=-0.00661946 0.00191632 8e-05 rpy=1.6673e-92 1.75162e-46 1.90372e-46; parent root -> part_1_1

File: models/wing_asy_right/urdf/wing_asy_right_visualizer.urdf (robot description, URDF)
Before this commit: robot wing_asy_right_visualizer, 3 links, 2 joints
Links:
- link part_1: geometry visual mesh filename=../meshes/Part_1.stl scale=100 100 100
- link part_1_1: geometry visual mesh filename=../meshes/Part_1_1.stl scale=100 100 100
Joints:
- removed joint group_1_fastened_joint
- added joint hanging_node_to_root_joint: type fixed, parent root, child part_1_1, origin xyz=0.186505 0.121117 0.0640399 rpy=-3.14159 1.99562e-30 -3.14159, axis 0 0 1
- joint fastened_1: child part_1_1 -> part_1; origin xyz=1.21431e-17 -2.81893e-18 -1.142e-33 rpy=-3.14159 -2.18953e-46 3.14159 -> xyz=-0.661946 0.191632 0.008 rpy=1.6673e-92 1.75162e-46 1.90372e-46; parent root -> part_1_1
