Commit message: Using the drake internal example (quadrotor meldis) instead of the external.

File: models/fwmav_asy/urdf/fwmav_asy.urdf (robot description, URDF)
Before this commit: robot fwmav_asy, 9 links, 8 joints
Links:
- added link left_wing_center_of_mass_marker; visual sphere radius=0.0001
- added link left_wing_support, mass 1e-09; collision cylinder length=0.0045 radius=5e-05; visual cylinder length=0.0045 radius=5e-05
- added link left_wing_support_pitch, mass 1e-09
- added link left_wing_support_yaw, mass 1e-09
- added link right_wing_support, mass 1e-09; collision cylinder length=0.0045 radius=5e-05; visual cylinder length=0.0045 radius=5e-05
- added link right_wing_support_pitch, mass 1e-09
- added link right_wing_support_yaw, mass 1e-09
Joints:
- added joint left_wing_center_of_mass_marker_joint: type fixed, parent left_wing_root, child left_wing_center_of_mass_marker, origin xyz=0 0 0 rpy=0 0 0
- added joint left_wing_support_joint: type fixed, parent left_wing_support_pitch, child left_wing_support, origin xyz=0.00200476 0 -0.00102148 rpy=0 2.04204 0
- added joint left_wing_support_pitch_joint: type revolute, parent left_wing_support_yaw, child left_wing_support_pitch, origin xyz=0 0 0 rpy=0 0 0, axis -1 0 0, limit lower=-1.5708 upper=1.5708 effort=1 velocity=100
- added joint left_wing_support_yaw_joint: type revolute, parent fuselage, child left_wing_support_yaw, origin xyz=0.00114 0 0.006675 rpy=0 0 0, axis 0 0 -1, limit lower=-1.5708 upper=1.5708 effort=1 velocity=100
- added joint right_wing_support_joint: type fixed, parent right_wing_support_pitch, child right_wing_support, origin xyz=-0.00200476 0 -0.00102148 rpy=0 -2.04204 0
- added joint right_wing_support_pitch_joint: type revolute, parent right_wing_support_yaw, child right_wing_support_pitch, origin xyz=0 0 0 rpy=0 0 0, axis 1 0 0, limit lower=-1.5708 upper=1.5708 effort=1 velocity=100
- added joint right_wing_support_yaw_joint: type revolute, parent fuselage, child right_wing_support_yaw, origin xyz=-0.00114 0 0.006675 rpy=0 0 0, axis 0 0 1, limit lower=-1.5708 upper=1.5708 effort=1 velocity=100
- joint left_wing_pitch_joint: axis 0 1 0 -> (none); limit lower=-1.5708 upper=1.5708 effort=1 velocity=100 -> (none); type revolute -> fixed
- joint left_wing_yaw_joint: axis 0 0 1 -> (none); limit lower=-1.5708 upper=1.5708 effort=1 velocity=100 -> (none); origin xyz=-0.00114 0.00114 0.006675 rpy=0 0 0 -> xyz=0.00940953 -0.000093 -0.00208996 rpy=0 0 0; parent fuselage -> left_wing_support_pitch; type revolute -> fixed
- joint right_wing_pitch_joint: axis 0 1 0 -> (none); limit lower=-1.5708 upper=1.5708 effort=1 velocity=100 -> (none); type revolute -> fixed
- joint right_wing_yaw_joint: axis 0 0 1 -> (none); limit lower=-1.5708 upper=1.5708 effort=1 velocity=100 -> (none); origin xyz=0.00114 -0.00114 0.006675 rpy=0 0 0 -> xyz=-0.00940953 -0.000093 -0.00208996 rpy=0 0 0; parent fuselage -> right_wing_support_pitch; type revolute -> fixed

File: models/wing_asy/urdf/wing_asy_visualizer.urdf (robot description, URDF)
Before this commit: robot wing_asy_visualizer, 3 links, 2 joints
Links:
- added link center_of_mass_marker; visual sphere radius=0.00015
Joints:
- added joint center_of_mass_marker_joint: type fixed, parent root, child center_of_mass_marker, origin xyz=0.00539918 -0.000922868 -4.71481e-05 rpy=0 0 0

Commit message: URDF just before adding more accurate hinge

File: models/fwmav_asy/urdf/fwmav_asy.urdf (robot description, URDF)
Before this commit: robot fwmav_asy, 16 links, 15 joints
Links:
- added link right_wing_center_marker; visual sphere radius=0.00015
- link right_wing_part_1: mass 8.16534e-11 -> 4.70198e-10
- link right_wing_part_1_1: mass 3.83835e-10 -> 8.16534e-11
Joints:
- removed joint left_wing_hanging_node_to_root_joint
- removed joint right_wing_hanging_node_to_root_joint
- added joint left_wing_fixed_node_to_root_joint: type fixed, parent left_wing_root, child left_wing_part_1, origin xyz=0.00122028 -0.000993447 -3.285e-05 rpy=0 0 0
- added joint right_wing_center_marker_joint: type fixed, parent right_wing_root, child right_wing_center_marker, origin xyz=0 0 0 rpy=0 0 0
- added joint right_wing_fixed_node_to_root_joint: type fixed, parent right_wing_root, child right_wing_part_1, origin xyz=0.0155574 0.00108164 -4.16358e-05 rpy=3.50068e-08 -1.35618e-08 -3.4518e-09
- joint left_wing_fastened_1: child left_wing_part_1 -> left_wing_part_1_1; origin xyz=-0.00679779 0.00217114 1.5e-06 rpy=0 0 0 -> xyz=-0.00661946 0.00191632 2.03288e-20 rpy=0 0 0; parent left_wing_part_1_1 -> left_wing_part_1
- joint left_wing_yaw_joint: origin xyz=0.00940953 -0.000093 -0.00208996 rpy=0 0 0 -> xyz=0.00940953 -0.000927 -0.00208996 rpy=0 0 0
- joint right_wing_fastened_1: child right_wing_part_1 -> right_wing_part_1_1; origin xyz=-0.00661946 0.00191632 8e-05 rpy=1.6673e-92 1.75162e-46 1.90372e-46 -> xyz=-0.010204 -0.000187856 3.97089e-18 rpy=2.11697e-49 -1.65436e-24 -2.55926e-25; parent right_wing_part_1_1 -> right_wing_part_1
- joint right_wing_yaw_joint: origin xyz=-0.00940953 -0.000093 -0.00208996 rpy=0 0 0 -> xyz=-0.00940953 -0.00089378 -0.00209934 rpy=0 0 0

File: models/wing_asy/urdf/wing_asy.urdf (robot description, URDF)
Before this commit: robot wing_asy, 3 links, 2 joints
Joints:
- removed joint fastened_2
- added joint fixed_node_to_root_joint: type fixed, parent root, child part_1, origin xyz=0.00122028 -0.000993447 -3.285e-05 rpy=0 -0 0, axis 0 0 1
- joint fastened_1: origin xyz=0 0 -8e-05 rpy=0 -0 0 -> xyz=-0.00661946 0.00191632 2.03288e-20 rpy=0 -0 0

File: models/wing_asy/urdf/wing_asy_visualizer.urdf (robot description, URDF)
Before this commit: robot wing_asy_visualizer, 4 links, 3 joints
Joints:
- removed joint fastened_2
- added joint fixed_node_to_root_joint: type fixed, parent root, child part_1, origin xyz=0.00122028 -0.000993447 -3.285e-05 rpy=0 -0 0, axis 0 0 1
- joint center_of_mass_marker_joint: origin xyz=0.00539918 -0.000922868 -4.71481e-05 rpy=0 0 0 -> xyz=0 0 0 rpy=0 0 0
- joint fastened_1: origin xyz=0 0 -8e-05 rpy=0 -0 0 -> xyz=-0.00661946 0.00191632 2.03288e-20 rpy=0 -0 0

File: models/wing_asy_right/urdf/wing_asy_right.urdf (robot description, URDF)
Before this commit: robot wing_asy_right, 3 links, 2 joints
Links:
- link part_1: mass 8.16534e-11 -> 4.70198e-10
- link part_1_1: mass 3.83835e-10 -> 8.16534e-11
Joints:
- removed joint group_1_fastened_joint
- added joint fixed_node_to_root_joint: type fixed, parent root, child part_1, origin xyz=0.0155574 0.00108164 -4.16358e-05 rpy=3.50068e-08 -1.35618e-08 -3.4518e-09, axis 0 0 1
- joint fastened_1: axis 0 0 -1 -> 0 0 1; origin xyz=1.21431e-17 -2.81893e-18 -1.142e-33 rpy=-3.14159 -2.18953e-46 3.14159 -> xyz=-0.010204 -0.000187856 3.97089e-18 rpy=2.11697e-49 -1.65436e-24 -2.55926e-25; parent root -> part_1

File: models/wing_asy_right/urdf/wing_asy_right_visualizer.urdf (robot description, URDF)
Before this commit: robot wing_asy_right_visualizer, 3 links, 2 joints
Links:
- link part_1: mass 8.16534e-11 -> 4.70198e-10
- link part_1_1: mass 3.83835e-10 -> 8.16534e-11
Joints:
- removed joint group_1_fastened_joint
- added joint fixed_node_to_root_joint: type fixed, parent root, child part_1, origin xyz=0.0155574 0.00108164 -4.16358e-05 rpy=3.50068e-08 -1.35618e-08 -3.4518e-09, axis 0 0 1
- joint fastened_1: axis 0 0 -1 -> 0 0 1; origin xyz=1.21431e-17 -2.81893e-18 -1.142e-33 rpy=-3.14159 -2.18953e-46 3.14159 -> xyz=-0.010204 -0.000187856 3.97089e-18 rpy=2.11697e-49 -1.65436e-24 -2.55926e-25; parent root -> part_1

Commit message: updated urdf

File: models/fwmav_asy/urdf/fwmav_asy.urdf (robot description, URDF)
Before this commit: robot fwmav_asy, 17 links, 16 joints
Links:
- removed link left_wing_support
- added link left_wing_support_base, mass 1e-09; collision cylinder length=0.00215 radius=5e-05; visual cylinder length=0.00215 radius=5e-05
- link left_wing_support_yaw: geometry collision cylinder length=0.00295204 radius=5e-05; visual cylinder length=0.00295204 radius=5e-05
Joints:
- removed joint left_wing_support_joint
- added joint left_wing_support_base_joint: type fixed, parent fuselage, child left_wing_support_base, origin xyz=0.00114 0 0.006675 rpy=0 0 0
- joint left_wing_support_pitch_joint: axis -1 0 0 -> 1 0 0; origin xyz=0 0 0 rpy=0 0 0 -> xyz=0.00293 0 -0.00036009 rpy=0 0 0
- joint left_wing_support_yaw_joint: axis 0 0 -1 -> 0 0 1; origin xyz=0.00114 0 0.006675 rpy=0 0 0 -> xyz=0.00215 0 0 rpy=0 0 0; parent fuselage -> left_wing_support_base
- joint left_wing_yaw_joint: origin xyz=0.00940953 -0.000927 -0.00208996 rpy=0 0 0 -> xyz=0 0 0 rpy=0 0 0
