Commit message: updated urdf with masses

File: models/robobee_assembly/urdf/robobee_assembly.urdf (robot description, URDF)
Before this commit: robot robobee_assembly_urdf, 36 links, 35 joints
Links:
- link hinge_base: mass 2.6141e-10 -> 4.18256e-07; geometry visual mesh filename=package://robobee_assembly/meshes/hinge_base.obj scale=1 1 1
- link hinge_wing: mass 3.20472e-10 -> 5.12755e-07; geometry visual mesh filename=package://robobee_assembly/meshes/hinge_wing.obj scale=1 1 1
- link part_1: mass 8.16534e-11 -> 7.68358e-08; geometry visual mesh filename=package://robobee_assembly/meshes/Part_1.obj scale=1 1 1
- link part_1_1: mass 3.83835e-10 -> 6.14136e-07; geometry visual mesh filename=package://robobee_assembly/meshes/Part_1_1.obj scale=1 1 1
- link part_1_2: mass 2.30323e-09 -> 3.68516e-06; geometry visual mesh filename=package://robobee_assembly/meshes/Part_1_2.obj scale=1 1 1
- link part_1_3: mass 2.52383e-09 -> 4.03812e-06; geometry visual mesh filename=package://robobee_assembly/meshes/Part_1_3.obj scale=1 1 1
- link part_1_4: mass 6.34231e-10 -> 1.01477e-06; geometry visual mesh filename=package://robobee_assembly/meshes/Part_1_4.obj scale=1 1 1
- link part_1_5: mass 1.06667e-09 -> 1.70668e-06; geometry visual mesh filename=package://robobee_assembly/meshes/Part_1_5.obj scale=1 1 1
- link part_1_6: mass 2.73911e-09 -> 4.38258e-06; geometry visual mesh filename=package://robobee_assembly/meshes/Part_1_6.obj scale=1 1 1
- link part_1_7: mass 8.16534e-11 -> 7.68358e-08; geometry visual mesh filename=package://robobee_assembly/meshes/Part_1.obj scale=1 1 1
- link part_1_8: mass 3.83835e-10 -> 6.14136e-07; geometry visual mesh filename=package://robobee_assembly/meshes/Part_1_1.obj scale=1 1 1
- link root: geometry visual mesh filename=package://robobee_assembly/meshes/hinge_base_Mirrored.obj scale=1 1 1; visual mesh filename=package://robobee_assembly/meshes/hinge_wing_Mirrored.obj scale=1 1 1
- link transmission_base: mass 7.30249e-10 -> 1.1684e-06; geometry visual mesh filename=package://robobee_assembly/meshes/transmission_base.obj scale=1 1 1
- link transmission_hinge: mass 6.98722e-10 -> 1.11796e-06; geometry visual mesh filename=package://robobee_assembly/meshes/transmission_hinge.obj scale=1 1 1
- link transmission_link_1: mass 1.84809e-10 -> 2.95694e-07; geometry visual mesh filename=package://robobee_assembly/meshes/transmission_link_1.obj scale=1 1 1
- link transmission_link_2: mass 8.6532e-11 -> 1.38451e-07; geometry visual mesh filename=package://robobee_assembly/meshes/transmission_link_2.obj scale=1 1 1
Joints:
- joint fastened_1: origin xyz=-0.000989203 0.000146549 1.5e-06 rpy=6.60706e-15 -3.11051e-15 -4.17166e-14 -> xyz=-0.000989203 0.000146549 1.5e-06 rpy=6.60706e-15 -3.11051e-15 -4.16889e-14
- joint fastened_2: origin xyz=-0.00301999 0.000805097 -0.0001175 rpy=3.14159 -1.61351e-27 1.2935e-26 -> xyz=-0.00301999 0.000805097 -0.0001175 rpy=3.14159 1.84962e-30 1.2935e-26
- joint hanging_node_to_root_joint: origin xyz=0.00488933 -0.000412 0.011418 rpy=1.5708 -2.03591e-15 1.20251e-11 -> xyz=0.00488933 -0.000412 0.011418 rpy=1.5708 -1.81387e-15 8.36974e-12
- joint revolute_1: origin xyz=-0.0106513 -7.98673e-05 -8e-05 rpy=3.14159 2.37887e-11 2.99451 -> xyz=-0.0106513 -7.98673e-05 -8e-05 rpy=3.14159 1.6557e-11 2.99451
- joint revolute_1_3: origin xyz=-0.00649814 -0.0104992 -0.000332133 rpy=-1.5708 -1.20251e-11 -0.147079 -> xyz=-0.00649814 -0.0104992 -0.000332133 rpy=-1.5708 -8.36975e-12 -0.147079
- joint revolute_1_4: origin xyz=0.000869661 9.99916e-05 -5.25e-05 rpy=-1.66533e-16 -2.77553e-17 1.41508e-24 -> xyz=0.000869661 9.99916e-05 -5.25e-05 rpy=-1.66533e-16 8.36971e-12 1.57362e-26
- joint revolute_1_5: origin xyz=0.00115694 0.000434896 -2.75e-05 rpy=-3.14237e-17 -1.61556e-27 3.9443e-31 -> xyz=0.00115694 0.000434896 -2.75e-05 rpy=-3.14237e-17 2.84992e-32 3.9443e-31
- joint revolute_1_6: origin xyz=0.000872592 -7.98673e-05 -1.0842e-19 rpy=7.21823e-17 -1.58803e-17 0.147079 -> xyz=0.000872592 -7.98673e-05 -5.42101e-20 rpy=7.21823e-17 -1.58803e-17 0.147079
- joint revolute_2_1: origin xyz=0.000136003 -9.03843e-14 -0.000403 rpy=1.11022e-16 5.36131e-11 -1.11022e-16 -> xyz=0.000136003 -9.03826e-14 -0.000403 rpy=-1.4376e-26 4.80874e-11 -2.41023e-26
- joint revolute_3_1: origin xyz=-0.0004 0 6.77626e-21 rpy=2.22045e-16 -5.36131e-11 -1.18673e-26 -> xyz=-0.0004 -1.73472e-18 -2.03288e-20 rpy=3.33067e-16 -5.64572e-11 -1.11022e-16

File: models/robobee_assembly/urdf/robobee_assembly_visualizer.urdf (robot description, URDF)
Before this commit: robot robobee_assembly_urdf, 36 links, 35 joints
Links:
- link hinge_base: geometry visual mesh filename=package://robobee_assembly/meshes/hinge_base.obj scale=1 1 1
- link hinge_wing: geometry visual mesh filename=package://robobee_assembly/meshes/hinge_wing.obj scale=1 1 1
- link part_1: geometry visual mesh filename=package://robobee_assembly/meshes/Part_1.obj scale=1 1 1
- link part_1_1: geometry visual mesh filename=package://robobee_assembly/meshes/Part_1_1.obj scale=1 1 1
- link part_1_2: geometry visual mesh filename=package://robobee_assembly/meshes/Part_1_2.obj scale=1 1 1
- link part_1_3: geometry visual mesh filename=package://robobee_assembly/meshes/Part_1_3.obj scale=1 1 1
- link part_1_4: geometry visual mesh filename=package://robobee_assembly/meshes/Part_1_4.obj scale=1 1 1
- link part_1_5: geometry visual mesh filename=package://robobee_assembly/meshes/Part_1_5.obj scale=1 1 1
- link part_1_6: geometry visual mesh filename=package://robobee_assembly/meshes/Part_1_6.obj scale=1 1 1
- link part_1_7: geometry visual mesh filename=package://robobee_assembly/meshes/Part_1.obj scale=1 1 1
- link part_1_8: geometry visual mesh filename=package://robobee_assembly/meshes/Part_1_1.obj scale=1 1 1
- link root: geometry visual mesh filename=package://robobee_assembly/meshes/hinge_base_Mirrored.obj scale=1 1 1; visual mesh filename=package://robobee_assembly/meshes/hinge_wing_Mirrored.obj scale=1 1 1
- link transmission_base: geometry visual mesh filename=package://robobee_assembly/meshes/transmission_base.obj scale=1 1 1
- link transmission_hinge: geometry visual mesh filename=package://robobee_assembly/meshes/transmission_hinge.obj scale=1 1 1
- link transmission_link_1: geometry visual mesh filename=package://robobee_assembly/meshes/transmission_link_1.obj scale=1 1 1
- link transmission_link_2: geometry visual mesh filename=package://robobee_assembly/meshes/transmission_link_2.obj scale=1 1 1
Joints:
- joint fastened_1: origin xyz=-0.000989203 0.000146549 1.5e-06 rpy=6.60706e-15 -3.11051e-15 -4.17166e-14 -> xyz=-0.000989203 0.000146549 1.5e-06 rpy=6.60706e-15 -3.11051e-15 -4.16889e-14
- joint fastened_2: origin xyz=-0.00301999 0.000805097 -0.0001175 rpy=3.14159 -1.61351e-27 1.2935e-26 -> xyz=-0.00301999 0.000805097 -0.0001175 rpy=3.14159 1.84962e-30 1.2935e-26
- joint hanging_node_to_root_joint: origin xyz=0.00488933 -0.000412 0.011418 rpy=1.5708 -2.03591e-15 1.20251e-11 -> xyz=0.00488933 -0.000412 0.011418 rpy=1.5708 -1.81387e-15 8.36974e-12
- joint revolute_1: origin xyz=-0.0106513 -7.98673e-05 -8e-05 rpy=3.14159 2.37887e-11 2.99451 -> xyz=-0.0106513 -7.98673e-05 -8e-05 rpy=3.14159 1.6557e-11 2.99451
- joint revolute_1_3: origin xyz=-0.00649814 -0.0104992 -0.000332133 rpy=-1.5708 -1.20251e-11 -0.147079 -> xyz=-0.00649814 -0.0104992 -0.000332133 rpy=-1.5708 -8.36975e-12 -0.147079
- joint revolute_1_4: origin xyz=0.000869661 9.99916e-05 -5.25e-05 rpy=-1.66533e-16 -2.77553e-17 1.41508e-24 -> xyz=0.000869661 9.99916e-05 -5.25e-05 rpy=-1.66533e-16 8.36971e-12 1.57362e-26
- joint revolute_1_5: origin xyz=0.00115694 0.000434896 -2.75e-05 rpy=-3.14237e-17 -1.61556e-27 3.9443e-31 -> xyz=0.00115694 0.000434896 -2.75e-05 rpy=-3.14237e-17 2.84992e-32 3.9443e-31
- joint revolute_1_6: origin xyz=0.000872592 -7.98673e-05 -1.0842e-19 rpy=7.21823e-17 -1.58803e-17 0.147079 -> xyz=0.000872592 -7.98673e-05 -5.42101e-20 rpy=7.21823e-17 -1.58803e-17 0.147079
- joint revolute_2_1: origin xyz=0.000136003 -9.03843e-14 -0.000403 rpy=1.11022e-16 5.36131e-11 -1.11022e-16 -> xyz=0.000136003 -9.03826e-14 -0.000403 rpy=-1.4376e-26 4.80874e-11 -2.41023e-26
- joint revolute_3_1: origin xyz=-0.0004 0 6.77626e-21 rpy=2.22045e-16 -5.36131e-11 -1.18673e-26 -> xyz=-0.0004 -1.73472e-18 -2.03288e-20 rpy=3.33067e-16 -5.64572e-11 -1.11022e-16
