Commit message: Revert "updates"
This reverts commit c64f437744879e22f18879df8d193bd6d5f11498.

File: models/robobee_assembly/urdf/robobee_assembly.urdf (robot description, URDF)
Before this commit: robot robobee_assembly, 32 links, 31 joints
Links:
- removed link hinge_base_1
- removed link hinge_wing_1
- removed link part_1_9
- removed link part_2
- removed link part_2_1
- removed link part_3
- removed link part_3__1__loop_closure
- removed link planar_2
- removed link planar_2_1
- removed link transmission_hinge__2__loop_closure
- removed link transmission_left_urdf__1_
- removed link transmission_right_urdf__1_
- added link hinge_base__1_, mass 1e-09
- added link hinge_wing__1_, mass 1e-09
- added link planar_1_2
- added link planar_1_3
- added link planar_2_loop_closure
- added link planar_2_loop_closure_1
- added link sketch_2__1_, mass 1e-09
- added link sketch_2__1__loop_closure, mass 1e-09
- added link sketch_3__1_, mass 1e-09
- added link transmission_base__1_, mass 1e-09
- added link transmission_hinge__2_, mass 1e-09
- added link transmission_hinge_mirrored__1_, mass 1e-09
- added link transmission_link_1__1_, mass 1e-09
- added link transmission_link_1__1__1, mass 1e-09
- added link transmission_link_2__1_, mass 1e-09
- added link transmission_urdf__1_
- link part_1_2: mass 2.95694e-07 -> 3.68516e-06
- link part_1_3: mass 3.68516e-06 -> 4.03812e-06
- link part_1_4: mass 4.03724e-06 -> 1.01477e-06
- link part_1_5: mass 1.01477e-06 -> 1.70668e-06
- link part_1_6: mass 1.70668e-06 -> 4.38258e-06
- link part_1_7: mass 4.38258e-06 -> 7.68358e-08; geometry visual mesh filename=package://robobee_assembly/meshes/Part_1.obj scale=1 1 1
- link part_1_8: mass 7.68358e-08 -> 6.14136e-07; geometry visual mesh filename=package://robobee_assembly/meshes/Part_1_1.obj scale=1 1 1
- link root: geometry visual mesh filename=package://robobee_assembly/meshes/hinge_base_Mirrored.obj scale=1 1 1; visual mesh filename=package://robobee_assembly/meshes/hinge_wing_Mirrored.obj scale=1 1 1
Joints:
- removed joint fastened_1_5
- removed joint fastened_3_1
- removed joint planar_2
- removed joint planar_2_1
- removed joint planar_2_2
- removed joint revolute_2_loop_closure
- removed joint revolute_2_loop_closure_1
- removed joint slider_2
- added joint group_1_fastened_joint_1: type fixed, parent sketch_3__1_, child sketch_2__1_, origin xyz=0 0 -2.1684e-19 rpy=-1.22762e-69 9.86076e-32 -2.48991e-38, axis 0 0 1
- added joint group_2_fastened_joint: type fixed, parent part_1_3, child sketch_3__1_, origin xyz=-0.000859972 -8.5e-05 -0.00856221 rpy=-1.22762e-69 9.86076e-32 -2.48991e-38, axis 0 0 1
- added joint hanging_node_to_root_joint: type fixed, parent root, child hinge_wing, origin xyz=0.00488933 -0.000412 0.011418 rpy=1.5708 -1.81387e-15 8.36974e-12, axis 0 0 1
- added joint planar_1_3: type prismatic, parent part_1_5, child planar_1_3, origin xyz=-0.00248559 0.000424 -0.000172 rpy=-1.5708 1.11022e-16 3.14159, axis 1 0 0, limit lower=-10000 upper=10000 effort=1 velocity=1
- added joint planar_1_4: type prismatic, parent planar_1_3, child planar_1_2, origin xyz=0 0 0 rpy=0 -0 0, axis 0 0 1, limit lower=-10000 upper=10000 effort=1 velocity=1
- added joint planar_1_5: type continuous, parent planar_1_2, child transmission_base, origin xyz=0 0 0 rpy=0 -0 0, axis 0 -1 0
- added joint planar_2_loop_closure: type prismatic, parent transmission_base, child planar_2_loop_closure_1, origin xyz=-0.000670593 0.00633515 -0.000434578 rpy=0 -1.5708 1.5708, axis 0 0 -1, limit lower=-10000 upper=10000 effort=1 velocity=1
- added joint planar_2_loop_closure_1: type prismatic, parent planar_2_loop_closure_1, child planar_2_loop_closure, origin xyz=0 0 0 rpy=0 -0 0, axis -1 0 0, limit lower=-10000 upper=10000 effort=1 velocity=1
- added joint planar_2_loop_closure_2: type continuous, parent planar_2_loop_closure, child sketch_2__1__loop_closure, origin xyz=0 0 0 rpy=0 -0 0, axis 0 1 0
- added joint revolute_1_5: type continuous, parent hinge_wing, child hinge_base, origin xyz=0.00115694 0.000434896 -2.75e-05 rpy=-3.14237e-17 2.84992e-32 3.9443e-31, axis 1 0 0
- added joint revolute_1_6: type continuous, parent hinge_wing, child part_1_8, origin xyz=0.000872592 -7.98673e-05 -5.42101e-20 rpy=7.21823e-17 -1.58803e-17 0.147079, axis 0 0 -1
- added joint revolute_2_1: type continuous, parent transmission_hinge, child transmission_link_2, origin xyz=0.000136003 -9.03826e-14 -0.000403 rpy=-1.4376e-26 4.80874e-11 -2.41023e-26, axis 0 -1 0
- joint fastened_1: axis 0 0 1 -> 0 0 -1; child airframe_asy__1_ -> part_1; origin xyz=0.000934002 2.68882e-17 -4.66478e-17 rpy=4.18096e-24 1.34417e-24 6.28657e-23 -> xyz=-0.000989203 0.000146549 1.5e-06 rpy=6.60706e-15 -3.11051e-15 -4.16889e-14; parent part_1_7 -> part_1_1
- joint fastened_1_1: axis 0 0 -1 -> 0 0 1; child part_1_5 -> transmission_urdf__1_; origin xyz=9.70117e-21 -6.53804e-21 6.09864e-20 rpy=-9.7945e-22 1.94289e-16 3.14159 -> xyz=-0.000670617 -3.84606e-08 0.000254 rpy=2.77556e-16 3.29303e-22 -2.22045e-16; parent root -> transmission_base
- joint fastened_1_2: axis 0 0 -1 -> 0 0 1; child part_1_8 -> airframe_asy__1_; origin xyz=-0.000989203 0.000146549 -8e-05 rpy=-5.93467e-15 1.27002e-15 1.98452e-15 -> xyz=0.000934002 2.95987e-17 -2.90837e-17 rpy=3.30872e-24 -3.37238e-29 6.58606e-23; parent part_1_9 -> part_1_6
- joint fastened_1_3: axis 0 0 1 -> 0 0 -1; child transmission_left_urdf__1_ -> part_1_4; origin xyz=0.00087 -0.000315038 0.0003645 rpy=-2.46517e-32 9.1608e-33 -1.12915e-64 -> xyz=6.39113e-20 0 0 rpy=7.77156e-16 3.87741e-26 -3.14159; parent transmission_base -> root
- joint fastened_1_4: axis 0 0 1 -> 0 0 -1; child transmission_right_urdf__1_ -> part_1_7; origin xyz=1.69673e-08 -0.000315057 -0.0003645 rpy=4.81906e-22 6.30258e-24 -3.87719e-26 -> xyz=-0.000989203 0.000146549 -8e-05 rpy=-5.93844e-15 1.27017e-15 1.98452e-15; parent part_2_1 -> part_1_8
- joint fastened_2: axis 1 0 0 -> -1 0 0; child hinge_base_1 -> transmission_hinge_mirrored__1_; origin xyz=0.000530962 0.00025 0.0001165 rpy=-3.14159 1.38778e-17 1.97215e-31 -> xyz=-0.00301999 0.000805097 -0.0001175 rpy=3.14159 1.84962e-30 1.2935e-26; parent part_2 -> hinge_base
- joint fastened_2_1: child part_1_4 -> part_1_3; origin xyz=0.001019 -8.5e-05 0.01037 rpy=-1.6075e-21 3.92469e-23 -1.5708 -> xyz=0.001019 -8.5e-05 0.01037 rpy=-1.11022e-16 -1.11022e-16 -1.5708; parent part_1_7 -> part_1_6
- joint fastened_3: child part_1_3 -> part_1_2; origin xyz=-0.00172 -2.17247e-17 3.46945e-18 rpy=3.59382e-23 1.6075e-21 -1.5708 -> xyz=-0.00172 3.70255e-17 6.93889e-17 rpy=-1.11022e-16 1.11022e-16 -1.5708; parent part_1_4 -> part_1_3
- joint fastened_4: child part_1_6 -> part_1_5; origin xyz=0.001794 -8.5e-05 0.01309 rpy=4.18096e-24 1.34417e-24 6.28657e-23 -> xyz=0.001794 -8.5e-05 0.01309 rpy=3.30872e-24 -3.37238e-29 6.58606e-23; parent part_1_7 -> part_1_6
- joint fastened_5: child part_1_7 -> part_1_6; origin xyz=0.000934 0.000775 9e-05 rpy=-3.30869e-24 -2.14693e-15 3.14159 -> xyz=0.000934 0.000775 9e-05 rpy=-3.30872e-24 -2.14693e-15 3.14159; parent part_1_5 -> part_1_4
- joint group_1_fastened_joint: origin xyz=-0.000859972 -8.5e-05 -0.00856221 rpy=-1.97215e-31 -3.64403e-37 3.15544e-30 -> xyz=-0.000859972 -8.5e-05 -0.00856221 rpy=-1.22762e-69 9.86076e-32 -2.48991e-38; parent part_1_4 -> part_1_3
- joint planar_1: axis 0 1 0 -> 1 0 0; mimic (none) -> joint=planar_1_3 multiplier=-1 offset=0; origin xyz=-0.0005345 0.00087 0.002233 rpy=-1.5708 1.11022e-16 1.5708 -> xyz=-0.00344588 -0.000219992 -0.012601 rpy=7.77156e-16 2.14693e-15 -6.58552e-22; parent part_1_4 -> part_1_5
- joint planar_1_1: axis 0 0 -1 -> 0 0 1; mimic (none) -> joint=planar_1_4 multiplier=1 offset=0
- joint planar_1_2: axis -1 0 0 -> 0 -1 0; child part_2_1 -> transmission_base__1_; mimic (none) -> joint=planar_1_5 multiplier=-1 offset=0
- joint revolute_1: axis 1 0 0 -> 0 0 -1; child hinge_wing_1 -> part_1_1; mimic (none) -> joint=revolute_1_6 multiplier=-1 offset=0; origin xyz=0.00301999 -0.000805097 0.0001175 rpy=-2.02606e-13 9.11904e-28 3.64615e-26 -> xyz=-0.0106513 -7.98673e-05 -8e-05 rpy=3.14159 1.6557e-11 2.99451; parent hinge_base_1 -> hinge_wing
- joint revolute_1_1: axis 0 0 -1 -> 0 -1 0; child part_1_9 -> transmission_hinge__2_; mimic (none) -> joint=revolute_1_4 multiplier=-1 offset=0; origin xyz=-0.000284345 -0.000514764 2.75e-05 rpy=7.18312e-17 -9.05233e-18 0.147079 -> xyz=0.000869661 9.99916e-05 -5.25e-05 rpy=0 -0 0; parent hinge_wing_1 -> transmission_base__1_
- joint revolute_1_2: axis 0 -1 0 -> 1 0 0; child transmission_hinge -> hinge_base__1_; mimic (none) -> joint=revolute_1_5 multiplier=-1 offset=0; origin xyz=0.00241028 -0.000215008 5.8e-05 rpy=3.33067e-16 4.78506e-14 2.22045e-16 -> xyz=0.000284345 0.000514764 -2.75e-05 rpy=0 -0 0; parent transmission_base -> hinge_wing__1_
- joint revolute_1_3: axis 0 -1 0 -> 0 0 -1; child part_2 -> hinge_wing__1_; origin xyz=0.00154034 -0.000215008 -5.8e-05 rpy=-1.17373e-16 -1.6523e-12 1.22465e-16 -> xyz=-0.00649814 -0.0104992 -0.000332133 rpy=-1.5708 -8.36975e-12 -0.147079; parent part_2_1 -> part_1_8
- joint revolute_1_4: axis 1 0 0 -> 0 -1 0; child hinge_wing -> transmission_hinge; origin xyz=0.00301999 -0.000805097 -1.25e-05 rpy=1.35891e-13 8.15236e-29 5.2262e-29 -> xyz=0.000869661 9.99916e-05 -5.25e-05 rpy=-1.66533e-16 8.36971e-12 1.57362e-26; parent hinge_base -> transmission_base
- joint revolute_2: axis 0 0 -1 -> 0 -1 0; child part_1_1 -> transmission_link_2__1_; mimic (none) -> joint=revolute_2_1 multiplier=-1 offset=0; origin xyz=-0.000284345 -0.000514764 2.75e-05 rpy=5.05422e-16 1.10012e-15 0.147079 -> xyz=0.000136003 -9.03854e-14 -0.000403 rpy=0 -0 0; parent hinge_wing -> transmission_hinge__2_
- joint revolute_3: child transmission_link_2 -> transmission_link_1__1_; mimic (none) -> joint=revolute_3_1 multiplier=-1 offset=0; origin xyz=0.000619747 -1.52279e-13 0.0001235 rpy=5.55112e-17 -3.87994e-13 1.94289e-16 -> xyz=-0.0004 0 0 rpy=0 -0 0; parent transmission_link_1 -> transmission_link_2__1_
- joint revolute_3_1: child part_3 -> transmission_link_1; origin xyz=0.000619747 -1.52281e-13 -0.0001235 rpy=-4.01838e-23 -5.29425e-13 1.22465e-16 -> xyz=-0.0004 -1.73472e-18 -2.03288e-20 rpy=3.33067e-16 -5.64572e-11 -1.11022e-16; parent part_1_2 -> transmission_link_2
- joint slider_1: axis -1 0 0 -> 1 8.23363e-12 0; child part_1_2 -> transmission_link_1__1__1; origin xyz=-0.001003 0.00152655 0.00244801 rpy=-1.5708 4.44089e-16 1.5708 -> xyz=-0.001003 0.00180136 0.00244801 rpy=1.5708 -3.15117e-11 1.5708; parent part_1_4 -> part_1_3

File: models/robobee_assembly/urdf/robobee_assembly_visualizer.urdf (robot description, URDF)
Before this commit: robot robobee_assembly, 32 links, 31 joints
Links:
- removed link hinge_base_1
- removed link hinge_wing_1
- removed link part_1_9
- removed link part_2
- removed link part_2_1
- removed link part_3
- removed link part_3__1__loop_closure
- removed link planar_2
- removed link planar_2_1
- removed link transmission_hinge__2__loop_closure
- removed link transmission_left_urdf__1_
- removed link transmission_right_urdf__1_
- added link hinge_base__1_
- added link hinge_wing__1_
- added link planar_1_2
- added link planar_1_3
- added link planar_2_loop_closure
- added link planar_2_loop_closure_1
- added link sketch_2__1_
- added link sketch_2__1__loop_closure
- added link sketch_3__1_
- added link transmission_base__1_
- added link transmission_hinge__2_
- added link transmission_hinge_mirrored__1_
- added link transmission_link_1__1_
- added link transmission_link_1__1__1
- added link transmission_link_2__1_
- added link transmission_urdf__1_
- link part_1_7: geometry visual mesh filename=package://robobee_assembly/meshes/Part_1.obj scale=1 1 1
- link part_1_8: geometry visual mesh filename=package://robobee_assembly/meshes/Part_1_1.obj scale=1 1 1
- link root: geometry visual mesh filename=package://robobee_assembly/meshes/hinge_base_Mirrored.obj scale=1 1 1; visual mesh filename=package://robobee_assembly/meshes/hinge_wing_Mirrored.obj scale=1 1 1
Joints:
- removed joint fastened_1_5
- removed joint fastened_3_1
- removed joint planar_2
- removed joint planar_2_1
- removed joint planar_2_2
- removed joint revolute_2_loop_closure
- removed joint revolute_2_loop_closure_1
- removed joint slider_2
- added joint group_1_fastened_joint_1: type fixed, parent sketch_3__1_, child sketch_2__1_, origin xyz=0 0 -2.1684e-19 rpy=-1.22762e-69 9.86076e-32 -2.48991e-38, axis 0 0 1
- added joint group_2_fastened_joint: type fixed, parent part_1_3, child sketch_3__1_, origin xyz=-0.000859972 -8.5e-05 -0.00856221 rpy=-1.22762e-69 9.86076e-32 -2.48991e-38, axis 0 0 1
- added joint hanging_node_to_root_joint: type fixed, parent root, child hinge_wing, origin xyz=0.00488933 -0.000412 0.011418 rpy=1.5708 -1.81387e-15 8.36974e-12, axis 0 0 1
- added joint planar_1_3: type prismatic, parent part_1_5, child planar_1_3, origin xyz=-0.00248559 0.000424 -0.000172 rpy=-1.5708 1.11022e-16 3.14159, axis 1 0 0, limit lower=-10000 upper=10000 effort=1 velocity=1
- added joint planar_1_4: type prismatic, parent planar_1_3, child planar_1_2, origin xyz=0 0 0 rpy=0 -0 0, axis 0 0 1, limit lower=-10000 upper=10000 effort=1 velocity=1
- added joint planar_1_5: type continuous, parent planar_1_2, child transmission_base, origin xyz=0 0 0 rpy=0 -0 0, axis 0 -1 0
- added joint planar_2_loop_closure: type prismatic, parent transmission_base, child planar_2_loop_closure_1, origin xyz=-0.000670593 0.00633515 -0.000434578 rpy=0 -1.5708 1.5708, axis 0 0 -1, limit lower=-10000 upper=10000 effort=1 velocity=1
- added joint planar_2_loop_closure_1: type prismatic, parent planar_2_loop_closure_1, child planar_2_loop_closure, origin xyz=0 0 0 rpy=0 -0 0, axis -1 0 0, limit lower=-10000 upper=10000 effort=1 velocity=1
- added joint planar_2_loop_closure_2: type continuous, parent planar_2_loop_closure, child sketch_2__1__loop_closure, origin xyz=0 0 0 rpy=0 -0 0, axis 0 1 0
- added joint revolute_1_5: type continuous, parent hinge_wing, child hinge_base, origin xyz=0.00115694 0.000434896 -2.75e-05 rpy=-3.14237e-17 2.84992e-32 3.9443e-31, axis 1 0 0
- added joint revolute_1_6: type continuous, parent hinge_wing, child part_1_8, origin xyz=0.000872592 -7.98673e-05 -5.42101e-20 rpy=7.21823e-17 -1.58803e-17 0.147079, axis 0 0 -1
- added joint revolute_2_1: type continuous, parent transmission_hinge, child transmission_link_2, origin xyz=0.000136003 -9.03826e-14 -0.000403 rpy=-1.4376e-26 4.80874e-11 -2.41023e-26, axis 0 -1 0
- joint fastened_1: axis 0 0 1 -> 0 0 -1; child airframe_asy__1_ -> part_1; origin xyz=0.000934002 2.68882e-17 -4.66478e-17 rpy=4.18096e-24 1.34417e-24 6.28657e-23 -> xyz=-0.000989203 0.000146549 1.5e-06 rpy=6.60706e-15 -3.11051e-15 -4.16889e-14; parent part_1_7 -> part_1_1
- joint fastened_1_1: axis 0 0 -1 -> 0 0 1; child part_1_5 -> transmission_urdf__1_; origin xyz=9.70117e-21 -6.53804e-21 6.09864e-20 rpy=-9.7945e-22 1.94289e-16 3.14159 -> xyz=-0.000670617 -3.84606e-08 0.000254 rpy=2.77556e-16 3.29303e-22 -2.22045e-16; parent root -> transmission_base
- joint fastened_1_2: axis 0 0 -1 -> 0 0 1; child part_1_8 -> airframe_asy__1_; origin xyz=-0.000989203 0.000146549 -8e-05 rpy=-5.93467e-15 1.27002e-15 1.98452e-15 -> xyz=0.000934002 2.95987e-17 -2.90837e-17 rpy=3.30872e-24 -3.37238e-29 6.58606e-23; parent part_1_9 -> part_1_6
- joint fastened_1_3: axis 0 0 1 -> 0 0 -1; child transmission_left_urdf__1_ -> part_1_4; origin xyz=0.00087 -0.000315038 0.0003645 rpy=-2.46517e-32 9.1608e-33 -1.12915e-64 -> xyz=6.39113e-20 0 0 rpy=7.77156e-16 3.87741e-26 -3.14159; parent transmission_base -> root
- joint fastened_1_4: axis 0 0 1 -> 0 0 -1; child transmission_right_urdf__1_ -> part_1_7; origin xyz=1.69673e-08 -0.000315057 -0.0003645 rpy=4.81906e-22 6.30258e-24 -3.87719e-26 -> xyz=-0.000989203 0.000146549 -8e-05 rpy=-5.93844e-15 1.27017e-15 1.98452e-15; parent part_2_1 -> part_1_8
- joint fastened_2: axis 1 0 0 -> -1 0 0; child hinge_base_1 -> transmission_hinge_mirrored__1_; origin xyz=0.000530962 0.00025 0.0001165 rpy=-3.14159 1.38778e-17 1.97215e-31 -> xyz=-0.00301999 0.000805097 -0.0001175 rpy=3.14159 1.84962e-30 1.2935e-26; parent part_2 -> hinge_base
- joint fastened_2_1: child part_1_4 -> part_1_3; origin xyz=0.001019 -8.5e-05 0.01037 rpy=-1.6075e-21 3.92469e-23 -1.5708 -> xyz=0.001019 -8.5e-05 0.01037 rpy=-1.11022e-16 -1.11022e-16 -1.5708; parent part_1_7 -> part_1_6
- joint fastened_3: child part_1_3 -> part_1_2; origin xyz=-0.00172 -2.17247e-17 3.46945e-18 rpy=3.59382e-23 1.6075e-21 -1.5708 -> xyz=-0.00172 3.70255e-17 6.93889e-17 rpy=-1.11022e-16 1.11022e-16 -1.5708; parent part_1_4 -> part_1_3
- joint fastened_4: child part_1_6 -> part_1_5; origin xyz=0.001794 -8.5e-05 0.01309 rpy=4.18096e-24 1.34417e-24 6.28657e-23 -> xyz=0.001794 -8.5e-05 0.01309 rpy=3.30872e-24 -3.37238e-29 6.58606e-23; parent part_1_7 -> part_1_6
- joint fastened_5: child part_1_7 -> part_1_6; origin xyz=0.000934 0.000775 9e-05 rpy=-3.30869e-24 -2.14693e-15 3.14159 -> xyz=0.000934 0.000775 9e-05 rpy=-3.30872e-24 -2.14693e-15 3.14159; parent part_1_5 -> part_1_4
- joint group_1_fastened_joint: origin xyz=-0.000859972 -8.5e-05 -0.00856221 rpy=-1.97215e-31 -3.64403e-37 3.15544e-30 -> xyz=-0.000859972 -8.5e-05 -0.00856221 rpy=-1.22762e-69 9.86076e-32 -2.48991e-38; parent part_1_4 -> part_1_3
- joint planar_1: axis 0 1 0 -> 1 0 0; mimic (none) -> joint=planar_1_3 multiplier=-1 offset=0; origin xyz=-0.0005345 0.00087 0.002233 rpy=-1.5708 1.11022e-16 1.5708 -> xyz=-0.00344588 -0.000219992 -0.012601 rpy=7.77156e-16 2.14693e-15 -6.58552e-22; parent part_1_4 -> part_1_5
- joint planar_1_1: axis 0 0 -1 -> 0 0 1; mimic (none) -> joint=planar_1_4 multiplier=1 offset=0
- joint planar_1_2: axis -1 0 0 -> 0 -1 0; child part_2_1 -> transmission_base__1_; mimic (none) -> joint=planar_1_5 multiplier=-1 offset=0
- joint revolute_1: axis 1 0 0 -> 0 0 -1; child hinge_wing_1 -> part_1_1; mimic (none) -> joint=revolute_1_6 multiplier=-1 offset=0; origin xyz=0.00301999 -0.000805097 0.0001175 rpy=-2.02606e-13 9.11904e-28 3.64615e-26 -> xyz=-0.0106513 -7.98673e-05 -8e-05 rpy=3.14159 1.6557e-11 2.99451; parent hinge_base_1 -> hinge_wing
- joint revolute_1_1: axis 0 0 -1 -> 0 -1 0; child part_1_9 -> transmission_hinge__2_; mimic (none) -> joint=revolute_1_4 multiplier=-1 offset=0; origin xyz=-0.000284345 -0.000514764 2.75e-05 rpy=7.18312e-17 -9.05233e-18 0.147079 -> xyz=0.000869661 9.99916e-05 -5.25e-05 rpy=0 -0 0; parent hinge_wing_1 -> transmission_base__1_
- joint revolute_1_2: axis 0 -1 0 -> 1 0 0; child transmission_hinge -> hinge_base__1_; mimic (none) -> joint=revolute_1_5 multiplier=-1 offset=0; origin xyz=0.00241028 -0.000215008 5.8e-05 rpy=3.33067e-16 4.78506e-14 2.22045e-16 -> xyz=0.000284345 0.000514764 -2.75e-05 rpy=0 -0 0; parent transmission_base -> hinge_wing__1_
- joint revolute_1_3: axis 0 -1 0 -> 0 0 -1; child part_2 -> hinge_wing__1_; origin xyz=0.00154034 -0.000215008 -5.8e-05 rpy=-1.17373e-16 -1.6523e-12 1.22465e-16 -> xyz=-0.00649814 -0.0104992 -0.000332133 rpy=-1.5708 -8.36975e-12 -0.147079; parent part_2_1 -> part_1_8
- joint revolute_1_4: axis 1 0 0 -> 0 -1 0; child hinge_wing -> transmission_hinge; origin xyz=0.00301999 -0.000805097 -1.25e-05 rpy=1.35891e-13 8.15236e-29 5.2262e-29 -> xyz=0.000869661 9.99916e-05 -5.25e-05 rpy=-1.66533e-16 8.36971e-12 1.57362e-26; parent hinge_base -> transmission_base
- joint revolute_2: axis 0 0 -1 -> 0 -1 0; child part_1_1 -> transmission_link_2__1_; mimic (none) -> joint=revolute_2_1 multiplier=-1 offset=0; origin xyz=-0.000284345 -0.000514764 2.75e-05 rpy=5.05422e-16 1.10012e-15 0.147079 -> xyz=0.000136003 -9.03854e-14 -0.000403 rpy=0 -0 0; parent hinge_wing -> transmission_hinge__2_
- joint revolute_3: child transmission_link_2 -> transmission_link_1__1_; mimic (none) -> joint=revolute_3_1 multiplier=-1 offset=0; origin xyz=0.000619747 -1.52279e-13 0.0001235 rpy=5.55112e-17 -3.87994e-13 1.94289e-16 -> xyz=-0.0004 0 0 rpy=0 -0 0; parent transmission_link_1 -> transmission_link_2__1_
- joint revolute_3_1: child part_3 -> transmission_link_1; origin xyz=0.000619747 -1.52281e-13 -0.0001235 rpy=-4.01838e-23 -5.29425e-13 1.22465e-16 -> xyz=-0.0004 -1.73472e-18 -2.03288e-20 rpy=3.33067e-16 -5.64572e-11 -1.11022e-16; parent part_1_2 -> transmission_link_2
- joint slider_1: axis -1 0 0 -> 1 8.23363e-12 0; child part_1_2 -> transmission_link_1__1__1; origin xyz=-0.001003 0.00152655 0.00244801 rpy=-1.5708 4.44089e-16 1.5708 -> xyz=-0.001003 0.00180136 0.00244801 rpy=1.5708 -3.15117e-11 1.5708; parent part_1_4 -> part_1_3
