Commit message: working flapping!

File: models/robobee_assembly/urdf/robobee_assembly.urdf (robot description, URDF)
Before this commit: robot robobee_assembly, 32 links, 31 joints
Links:
- removed link part_1_9
- removed link part_2
- removed link part_2_1
- removed link part_3
- removed link part_3__1__loop_closure
- removed link planar_1
- removed link planar_1_1
- removed link planar_2
- removed link planar_2_1
- removed link transmission_hinge__2__loop_closure
- added link part_1__1__loop_closure, mass 1e-09
- added link part_1__2__loop_closure, mass 1e-09
- added link planar_1_loop_closure
- added link planar_1_loop_closure_1
- added link planar_2_loop_closure
- added link planar_2_loop_closure_1
- added link transmission_base__1__loop_closure, mass 1e-09
- added link transmission_link_2__1__loop_closure, mass 1e-09
- added link transmission_right_link_1, mass 2.95694e-07; visual mesh filename=package://robobee_assembly/meshes/transmission_right_link_1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 scale=1 1 1
- added link transmission_right_link_2, mass 1.38451e-07; visual mesh filename=package://robobee_assembly/meshes/transmission_right_link_2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 scale=1 1 1
- added link transmission_right_link_2__1__loop_closure, mass 1e-09
- added link transmission_right_link_base, mass 1.16841e-06; visual mesh filename=package://robobee_assembly/meshes/transmission_right_link_b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 scale=1 1 1
- added link transmission_right_link_base__2__loop_closure, mass 1e-09
- added link transmission_right_link_hinge, mass 1.11797e-06; visual mesh filename=package://robobee_assembly/meshes/transmission_right_link_h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 scale=1 1 1
- link part_1_2: mass 2.95694e-07 -> 3.68516e-06
- link part_1_3: mass 3.68516e-06 -> 4.03724e-06
- link part_1_4: mass 4.03724e-06 -> 1.01477e-06
- link part_1_5: mass 1.01477e-06 -> 1.70668e-06
- link part_1_6: mass 1.70668e-06 -> 4.38258e-06
- link part_1_7: mass 4.38258e-06 -> 7.68358e-08; geometry visual mesh filename=package://robobee_assembly/meshes/Part_1.obj scale=1 1 1
- link part_1_8: mass 7.68358e-08 -> 6.14136e-07; geometry visual mesh filename=package://robobee_assembly/meshes/Part_1_1.obj scale=1 1 1
Joints:
- removed joint fastened_2_1
- removed joint fastened_3_1
- removed joint fastened_4
- removed joint fastened_5
- removed joint planar_1
- removed joint planar_1_1
- removed joint planar_1_2
- removed joint planar_2
- removed joint planar_2_1
- removed joint planar_2_2
- added joint fastened_3_loop_closure: type fixed, parent part_1_3, child part_1__1__loop_closure, origin xyz=-0.000860028 8.5e-05 0.00856221 rpy=3.59382e-23 1.6075e-21 -1.5708, axis 0 0 1
- added joint fastened_4_loop_closure: type fixed, parent part_1_5, child part_1__2__loop_closure, origin xyz=0.00086 -0.0005575 -8.5e-05 rpy=-4.18096e-24 -1.34417e-24 -6.28657e-23, axis 0 0 1
- added joint fixed_node_to_root_joint: type fixed, parent root, child part_1_6, origin xyz=2.0772e-09 -0.000775 -0.00011 rpy=9.76141e-22 -2.34122e-15 -2.22045e-16, axis 0 0 1
- added joint fixed_node_to_root_joint_1: type fixed, parent root, child part_1_2, origin xyz=2.0772e-09 0.000775 0.0066775 rpy=-9.7945e-22 2.34122e-15 3.14159, axis 0 0 1
- added joint fixed_node_to_root_joint_2: type fixed, parent root, child part_1_5, origin xyz=2.0772e-09 -0.0003025 0.013265 rpy=9.80322e-22 -2.34122e-15 -2.22045e-16, axis 0 0 1
- added joint fixed_node_to_root_joint_3: type fixed, parent root, child part_1_3, origin xyz=2.0772e-09 -2.75209e-08 0.00189779 rpy=2.34122e-15 1.9429e-16 -1.5708, axis 0 0 1
- added joint fixed_node_to_root_joint_4: type fixed, parent root, child transmission_base, origin xyz=-0.00421149 0.000143 0.011928 rpy=-1.5708 2.31347e-15 3.14159, axis 0 0 1
- added joint fixed_node_to_root_joint_5: type fixed, parent root, child transmission_right_link_base, origin xyz=0.00252376 -0.000639387 0.0123379 rpy=-1.5708 -2.14693e-15 -2.55351e-14, axis 0 0 1
- added joint planar_1_loop_closure: type prismatic, parent part_1_3, child planar_1_loop_closure_1, origin xyz=0.000325472 0.000955 0.0107952 rpy=-1.5708 1.11022e-16 1.5708, axis 0 1 0, limit lower=-10000 upper=10000 effort=1 velocity=1
- added joint planar_1_loop_closure_1: type prismatic, parent planar_1_loop_closure_1, child planar_1_loop_closure, origin xyz=0 0 0 rpy=0 -0 0, axis 0 0 -1, limit lower=-10000 upper=10000 effort=1 velocity=1
- added joint planar_1_loop_closure_2: type continuous, parent planar_1_loop_closure, child transmission_right_link_base__2__loop_closure, origin xyz=0 0 0 rpy=0 -0 0, axis -1 0 0
- added joint planar_2_loop_closure: type prismatic, parent part_1_3, child planar_2_loop_closure_1, origin xyz=0.000325472 -8.5e-05 0.0107952 rpy=-1.5708 -0 -1.5708, axis 0 0 1, limit lower=-10000 upper=10000 effort=1 velocity=1
- added joint planar_2_loop_closure_1: type prismatic, parent planar_2_loop_closure_1, child planar_2_loop_closure, origin xyz=0 0 0 rpy=0 -0 0, axis 0 -1 0, limit lower=-10000 upper=10000 effort=1 velocity=1
- added joint planar_2_loop_closure_2: type continuous, parent planar_2_loop_closure, child transmission_base__1__loop_closure, origin xyz=0 0 0 rpy=0 -0 0, axis 1 0 0
- joint fastened_1: origin xyz=0.000934002 2.68882e-17 -4.66478e-17 rpy=4.18096e-24 1.34417e-24 6.28657e-23 -> xyz=4.29387e-19 2.68882e-17 0.0002 rpy=4.18096e-24 1.34417e-24 6.28657e-23; parent part_1_7 -> part_1_6
- joint fastened_1_1: child part_1_5 -> part_1_4
- joint fastened_1_2: child part_1_8 -> part_1_7; parent part_1_9 -> part_1_8
- joint fastened_1_3: origin xyz=0.00087 -0.000315038 0.0003645 rpy=-2.46517e-32 9.1608e-33 -1.12915e-64 -> xyz=-0.0032565 -0.00108003 0.000833 rpy=-2.46517e-32 9.1608e-33 -1.12915e-64
- joint fastened_1_4: origin xyz=1.69673e-08 -0.000315057 -0.0003645 rpy=4.81906e-22 6.30258e-24 -3.87719e-26 -> xyz=-0.00156874 -0.000670143 -5.06127e-05 rpy=4.81906e-22 6.30258e-24 -3.87719e-26; parent part_2_1 -> transmission_right_link_base
- joint fastened_2: parent part_2 -> transmission_right_link_hinge
- joint fastened_3: axis 0 0 1 -> 1 0 0; child part_1_3 -> hinge_base; origin xyz=-0.00172 -2.17247e-17 3.46945e-18 rpy=3.59382e-23 1.6075e-21 -1.5708 -> xyz=0.000531022 0.00025 -0.0001165 rpy=3.14159 -3.83103e-16 -5.09355e-16; parent part_1_4 -> transmission_hinge
- joint group_1_fastened_joint: origin xyz=-0.000859972 -8.5e-05 -0.00856221 rpy=-1.97215e-31 -3.64403e-37 3.15544e-30 -> xyz=-3.30872e-24 0 -2.1684e-19 rpy=-1.97215e-31 -3.64403e-37 3.15544e-30; parent part_1_4 -> part_1_3
- joint revolute_1: origin xyz=0.00301999 -0.000805097 0.0001175 rpy=-2.02606e-13 9.11904e-28 3.64615e-26 -> xyz=0.00301999 -0.000805097 0.0001175 rpy=-2.02723e-13 8.23461e-28 3.64631e-26
- joint revolute_1_1: child part_1_9 -> part_1_8
- joint revolute_1_2: origin xyz=0.00241028 -0.000215008 5.8e-05 rpy=3.33067e-16 4.78506e-14 2.22045e-16 -> xyz=-0.00171622 -0.00098 0.0005265 rpy=3.33067e-16 4.78506e-14 2.22045e-16
- joint revolute_1_3: child part_2 -> transmission_right_link_hinge; origin xyz=0.00154034 -0.000215008 -5.8e-05 rpy=-1.17373e-16 -1.6523e-12 1.22465e-16 -> xyz=-2.84212e-05 -0.000570095 0.000255887 rpy=-4.87542e-22 -1.51459e-12 2.58466e-26; parent part_2_1 -> transmission_right_link_base
- joint revolute_2_loop_closure: child transmission_hinge__2__loop_closure -> transmission_link_2__1__loop_closure; origin xyz=0.0004 0 2.03288e-20 rpy=2.90892e-30 4.10504e-13 -6.7842e-29 -> xyz=0.000136003 -9.03843e-14 -0.000403 rpy=-2.95823e-30 -4.10504e-13 6.70532e-29; parent transmission_link_2 -> transmission_hinge
- joint revolute_2_loop_closure_1: child part_3__1__loop_closure -> transmission_right_link_2__1__loop_closure; origin xyz=0.000135962 -1.10413e-13 0.000403 rpy=-3.32479e-24 1.12288e-12 -3.94432e-31 -> xyz=0.000135962 -1.10413e-13 0.000403 rpy=-3.32479e-24 1.10071e-12 -4.33874e-30; parent part_2 -> transmission_right_link_hinge
- joint revolute_3_1: child part_3 -> transmission_right_link_2; origin xyz=0.000619747 -1.52281e-13 -0.0001235 rpy=-4.01838e-23 -5.29425e-13 1.22465e-16 -> xyz=0.000619747 -1.52281e-13 -0.0001235 rpy=1.17373e-16 -4.13882e-13 3.87167e-26; parent part_1_2 -> transmission_right_link_1
- joint slider_1: child part_1_2 -> transmission_right_link_1; origin xyz=-0.001003 0.00152655 0.00244801 rpy=-1.5708 4.44089e-16 1.5708 -> xyz=-0.000143028 0.00161155 0.0110102 rpy=-1.5708 4.44089e-16 1.5708; parent part_1_4 -> part_1_3
- joint slider_2: origin xyz=-0.001003 -0.00169653 0.00244801 rpy=-1.5708 3.33067e-16 -1.5708 -> xyz=-0.000143028 -0.00161153 0.0110102 rpy=-1.5708 3.33067e-16 -1.5708; parent part_1_4 -> part_1_3

Commit message: kinematic visualize_robobee_linkage written

File: models/robobee_assembly/urdf/robobee_assembly.urdf (robot description, URDF)
Before this commit: robot robobee_assembly, 36 links, 35 joints
Links:
- removed link hinge_base_1
- removed link hinge_wing_1
- removed link part_1_7
- removed link part_1_8
- removed link planar_1_loop_closure
- removed link planar_1_loop_closure_1
- removed link planar_2_loop_closure
- removed link planar_2_loop_closure_1
- removed link transmission_base__1__loop_closure
- removed link transmission_right_link_base__2__loop_closure
- added link hinge_right_base, mass 4.17643e-07; visual mesh filename=package://robobee_assembly/meshes/hinge_right_base.obj scale=1 1 1
- added link hinge_right_wing, mass 5.141e-07; visual mesh filename=package://robobee_assembly/meshes/hinge_right_wing.obj scale=1 1 1
- added link wing_asy__1_
- added link wing_asy__2_
- added link wing_cf, mass 6.14136e-07; visual mesh filename=package://robobee_assembly/meshes/wing_cf.obj scale=1 1 1
- added link wing_cf_1, mass 6.14136e-07; visual mesh filename=package://robobee_assembly/meshes/wing_cf.obj scale=1 1 1
- link part_1_1: mass 6.14136e-07 -> 3.68516e-06
- link part_1_2: mass 3.68516e-06 -> 4.03724e-06
- link part_1_3: mass 4.03724e-06 -> 1.01477e-06
- link part_1_4: mass 1.01477e-06 -> 1.70668e-06
- link part_1_5: mass 1.70668e-06 -> 4.38258e-06
- link part_1_6: mass 4.38258e-06 -> 7.68358e-08; geometry visual mesh filename=package://robobee_assembly/meshes/Part_1.obj scale=1 1 1
Joints:
- removed joint fastened_3
- removed joint planar_1_loop_closure
- removed joint planar_1_loop_closure_1
- removed joint planar_1_loop_closure_2
- removed joint planar_2_loop_closure
- removed joint planar_2_loop_closure_1
- removed joint planar_2_loop_closure_2
- added joint fixed_node_to_root_joint_6: type fixed, parent root, child transmission_right_link_base, origin xyz=0.00252376 -0.000639387 0.0123379 rpy=-1.5708 -2.14693e-15 -2.55351e-14, axis 0 0 1
- added joint revolute_1_5: type continuous, parent transmission_right_link_base, child transmission_right_link_hinge, origin xyz=-2.84212e-05 -0.000570095 0.000255887 rpy=-4.87542e-22 -1.51459e-12 2.58466e-26, axis -0 1 -0
- added joint revolute_1_6: type fixed, parent wing_cf, child wing_asy__2_, origin xyz=8.67362e-19 1.73472e-18 8e-05 rpy=1.69776e-17 7.48642e-17 -4.16334e-17, axis 0 0 1
- joint fastened_1: parent part_1_6 -> part_1_5
- joint fastened_1_1: axis 0 0 -1 -> -0 -0 1; child part_1_4 -> part_1_6; origin xyz=9.70117e-21 -6.53804e-21 6.09864e-20 rpy=-9.7945e-22 1.94289e-16 3.14159 -> xyz=-0.000989203 0.000146549 -8e-05 rpy=-1.78763e-15 -1.24258e-16 -5.27356e-16; parent root -> wing_cf_1
- joint fastened_1_2: axis 0 0 -1 -> -1 -0 -0; child part_1_7 -> hinge_right_base; origin xyz=-0.000989203 0.000146549 -8e-05 rpy=-5.93467e-15 1.27002e-15 1.98452e-15 -> xyz=0.000531022 0.00025 -0.0001165 rpy=3.14159 8.58946e-17 1.80013e-17; parent part_1_8 -> transmission_hinge
- joint fastened_1_3: axis 0 0 1 -> -0 -0 -1
- joint fastened_1_4: axis 0 0 1 -> -0 -0 -1
- joint fastened_1_5: child part_1 -> wing_cf; origin xyz=-0.000989203 0.000146549 -8e-05 rpy=3.28429e-47 -4.73317e-30 -1.38778e-17 -> xyz=-0.001 -5.20417e-18 1.5e-06 rpy=-3.44846e-15 9.19263e-16 0.147079; parent part_1_1 -> part_1
- joint fastened_2: axis 1 0 0 -> -1 -0 -0; child hinge_base_1 -> hinge_base
- joint fastened_3_loop_closure: parent part_1_3 -> part_1_2
- joint fastened_4_loop_closure: parent part_1_5 -> part_1_4
- joint fixed_node_to_root_joint: child part_1_6 -> part_1_3; origin xyz=2.0772e-09 -0.000775 -0.00011 rpy=9.76141e-22 -2.34122e-15 -2.22045e-16 -> xyz=-3.12792e-17 1.40187e-16 4.5e-05 rpy=-9.7945e-22 1.94289e-16 3.14159
- joint fixed_node_to_root_joint_1: child part_1_2 -> part_1_5; origin xyz=2.0772e-09 0.000775 0.0066775 rpy=-9.7945e-22 2.34122e-15 3.14159 -> xyz=2.0772e-09 -0.000775 -0.00011 rpy=9.76141e-22 -2.34122e-15 -2.22045e-16
- joint fixed_node_to_root_joint_2: child part_1_5 -> part_1_1; origin xyz=2.0772e-09 -0.0003025 0.013265 rpy=9.80322e-22 -2.34122e-15 -2.22045e-16 -> xyz=2.0772e-09 0.000775 0.0066775 rpy=-9.7945e-22 2.34122e-15 3.14159
- joint fixed_node_to_root_joint_3: child part_1_3 -> part_1_4; origin xyz=2.0772e-09 -2.75209e-08 0.00189779 rpy=2.34122e-15 1.9429e-16 -1.5708 -> xyz=2.0772e-09 -0.0003025 0.013265 rpy=9.80322e-22 -2.34122e-15 -2.22045e-16
- joint fixed_node_to_root_joint_4: child transmission_base -> part_1_2; origin xyz=-0.00421149 0.000143 0.011928 rpy=-1.5708 2.31347e-15 3.14159 -> xyz=2.0772e-09 -2.75209e-08 0.00189779 rpy=2.34122e-15 1.9429e-16 -1.5708
- joint fixed_node_to_root_joint_5: child transmission_right_link_base -> transmission_base; origin xyz=0.00252376 -0.000639387 0.0123379 rpy=-1.5708 -2.14693e-15 -2.55351e-14 -> xyz=-0.00421149 0.000143 0.011928 rpy=-1.5708 2.31347e-15 3.14159
- joint group_1_fastened_joint: axis 0 0 1 -> -0 -0 -1; parent part_1_3 -> part_1_2
- joint revolute_1: child hinge_wing_1 -> hinge_wing; origin xyz=0.00301999 -0.000805097 0.0001175 rpy=-2.02723e-13 8.23461e-28 3.64631e-26 -> xyz=0.00301999 -0.000805097 0.0001175 rpy=1.79153e-10 2.24404e-17 2.26168e-16; parent hinge_base_1 -> hinge_base
- joint revolute_1_1: axis 0 0 -1 -> 0 0 1; child part_1_8 -> wing_asy__1_; origin xyz=-0.000284345 -0.000514764 2.75e-05 rpy=7.18312e-17 -9.05233e-18 0.147079 -> xyz=-0.000989203 0.000146549 5.42101e-20 rpy=-1.49813e-18 -7.00953e-16 -0.147079; parent hinge_wing_1 -> wing_cf_1; type continuous -> fixed
- joint revolute_1_2: axis 0 -1 0 -> -0 -0 1; child transmission_hinge -> wing_cf_1; limit (none) -> lower=0 upper=0 effort=1 velocity=1; origin xyz=-0.00171622 -0.00098 0.0005265 rpy=3.33067e-16 4.78506e-14 2.22045e-16 -> xyz=-0.000284345 -0.000514764 2.75e-05 rpy=3.47914e-17 4.2275e-16 0.147079; parent transmission_base -> hinge_wing; type continuous -> revolute
- joint revolute_1_3: axis 0 -1 0 -> 1 0 0; child transmission_right_link_hinge -> hinge_right_wing; origin xyz=-2.84212e-05 -0.000570095 0.000255887 rpy=-4.87542e-22 -1.51459e-12 2.58466e-26 -> xyz=0.00301999 -0.000805 -0.000105 rpy=-5.55112e-17 2.77556e-17 -2.77556e-17; parent transmission_right_link_base -> hinge_right_base
- joint revolute_1_4: axis 1 0 0 -> -0 1 -0; child hinge_wing -> transmission_hinge; origin xyz=0.00301999 -0.000805097 -1.25e-05 rpy=1.35891e-13 8.15236e-29 5.2262e-29 -> xyz=-0.00171622 -0.00098 0.0005265 rpy=3.33067e-16 4.78506e-14 2.22045e-16; parent hinge_base -> transmission_base
- joint revolute_2: child part_1_1 -> part_1; limit (none) -> lower=0 upper=0 effort=1 velocity=1; origin xyz=-0.000284345 -0.000514764 2.75e-05 rpy=5.05422e-16 1.10012e-15 0.147079 -> xyz=-0.000294368 -0.000524845 -4e-05 rpy=4.08631e-15 -3.63443e-16 1.76248e-15; parent hinge_wing -> hinge_right_wing; type continuous -> revolute
- joint revolute_2_loop_closure: axis 0 -1 0 -> -0 1 -0
- joint revolute_2_loop_closure_1: axis 0 -1 0 -> -0 1 -0
- joint revolute_3: axis 0 -1 0 -> -0 1 -0
- joint slider_1: parent part_1_3 -> part_1_2
- joint slider_2: parent part_1_3 -> part_1_2

Commit message: left wing works!

File: models/robobee_assembly/urdf/robobee_assembly.urdf (robot description, URDF)
Before this commit: robot robobee_assembly, 32 links, 31 joints
Joints:
- joint revolute_1_3: limit (none) -> lower=-0.523599 upper=0.523599 effort=1 velocity=1
- joint revolute_1_4: limit (none) -> lower=-0.523599 upper=0.523599 effort=1 velocity=1

Commit message: updated urdf with latest

File: models/robobee_assembly/urdf/robobee_assembly.urdf (robot description, URDF)
Before this commit: robot robobee_assembly, 32 links, 31 joints
Links:
- removed link hinge_base
- removed link hinge_wing
- removed link part_1_5
- removed link part_1_6
- removed link wing_asy__2_
- added link hinge_left_base, mass 4.17643e-07; visual mesh filename=package://robobee_assembly/meshes/hinge_left_base.obj scale=1 1 1
- added link hinge_left_wing, mass 5.141e-07; visual mesh filename=package://robobee_assembly/meshes/hinge_left_wing.obj scale=1 1 1
- added link wing_asy_right__1_
- added link wing_membrane, mass 7.68358e-08; visual mesh filename=package://robobee_assembly/meshes/wing_membrane.obj scale=1 1 1
- added link wing_membrane_1, mass 7.68358e-08; visual mesh filename=package://robobee_assembly/meshes/wing_membrane.obj scale=1 1 1
- link hinge_right_base: mass 4.17643e-07 -> 4.18256e-07
- link hinge_right_wing: mass 5.141e-07 -> 5.12755e-07
- link part_1: mass 7.68358e-08 -> 3.68516e-06
- link part_1_1: mass 3.68516e-06 -> 4.03724e-06
- link part_1_2: mass 4.03724e-06 -> 1.01477e-06
- link part_1_3: mass 1.01477e-06 -> 1.70668e-06
- link part_1_4: mass 1.70668e-06 -> 4.38258e-06
Joints:
- removed joint revolute_1_5
- removed joint revolute_1_6
- added joint fastened_2_1: type fixed, parent wing_cf_1, child wing_asy__1_, origin xyz=-0.000989203 0.000146549 0 rpy=1.87477e-15 -9.72416e-17 -5.68989e-16, axis -0 -0 -1
- added joint fastened_2_2: type fixed, parent wing_cf, child wing_asy_right__1_, origin xyz=0.0050447 -0.000818183 -8.67362e-19 rpy=-3.14159 4.54119e-29 -3.14159, axis 0 0 1
- joint fastened_1: parent part_1_5 -> part_1_4
- joint fastened_1_1: child part_1_6 -> wing_membrane_1
- joint fastened_1_2: child hinge_right_base -> hinge_left_base; origin xyz=0.000531022 0.00025 -0.0001165 rpy=3.14159 8.58946e-17 1.80013e-17 -> xyz=0.000531022 0.00025 -0.0001165 rpy=-3.14159 -6.93889e-17 2.55651e-17
- joint fastened_1_5: child wing_cf -> wing_membrane; origin xyz=-0.001 -5.20417e-18 1.5e-06 rpy=-3.44846e-15 9.19263e-16 0.147079 -> xyz=-0.000247301 3.66373e-05 8e-05 rpy=4.16334e-17 -3.88578e-16 -1.92593e-33; parent part_1 -> wing_cf
- joint fastened_2: child hinge_base -> hinge_right_base
- joint fastened_3_loop_closure: parent part_1_2 -> part_1_1
- joint fastened_4_loop_closure: parent part_1_4 -> part_1_3
- joint fixed_node_to_root_joint: child part_1_3 -> part_1_2
- joint fixed_node_to_root_joint_1: child part_1_5 -> part_1_4
- joint fixed_node_to_root_joint_2: child part_1_1 -> part_1
- joint fixed_node_to_root_joint_3: child part_1_4 -> part_1_3
- joint fixed_node_to_root_joint_4: child part_1_2 -> part_1_1
- joint group_1_fastened_joint: parent part_1_2 -> part_1_1
- joint revolute_1: child hinge_wing -> hinge_right_wing; parent hinge_base -> hinge_right_base
- joint revolute_1_1: axis 0 0 1 -> -0 -0 1; child wing_asy__1_ -> wing_cf_1; limit (none) -> lower=0 upper=0 effort=1 velocity=1; origin xyz=-0.000989203 0.000146549 5.42101e-20 rpy=-1.49813e-18 -7.00953e-16 -0.147079 -> xyz=-0.000284345 -0.000514764 2.75e-05 rpy=3.47914e-17 4.2275e-16 0.147079; parent wing_cf_1 -> hinge_right_wing; type fixed -> revolute
- joint revolute_1_2: axis -0 -0 1 -> 1 0 0; child wing_cf_1 -> hinge_left_wing; limit lower=0 upper=0 effort=1 velocity=1 -> (none); origin xyz=-0.000284345 -0.000514764 2.75e-05 rpy=3.47914e-17 4.2275e-16 0.147079 -> xyz=0.00301999 -0.000805 -0.000105 rpy=-4.16026e-16 1.11022e-16 6.0408e-17; parent hinge_wing -> hinge_left_base; type revolute -> continuous
- joint revolute_1_3: axis 1 0 0 -> -0 1 -0; child hinge_right_wing -> transmission_hinge; origin xyz=0.00301999 -0.000805 -0.000105 rpy=-5.55112e-17 2.77556e-17 -2.77556e-17 -> xyz=-0.00171622 -0.00098 0.0005265 rpy=-1.83873e-16 -5.36779e-13 2.71791e-17; parent hinge_right_base -> transmission_base; type continuous -> revolute
- joint revolute_1_4: child transmission_hinge -> transmission_right_link_hinge; origin xyz=-0.00171622 -0.00098 0.0005265 rpy=3.33067e-16 4.78506e-14 2.22045e-16 -> xyz=-2.84212e-05 -0.000570095 0.000255887 rpy=-4.87542e-22 -1.51459e-12 2.58466e-26; parent transmission_base -> transmission_right_link_base; type continuous -> revolute
- joint revolute_2: axis 0 0 -1 -> -0 -0 -1; child part_1 -> wing_cf; origin xyz=-0.000294368 -0.000524845 -4e-05 rpy=4.08631e-15 -3.63443e-16 1.76248e-15 -> xyz=-0.00103581 -0.000520981 -7.6896e-06 rpy=4.59944e-18 -2.81431e-17 0.147079; parent hinge_right_wing -> hinge_left_wing
- joint revolute_2_loop_closure: origin xyz=0.000136003 -9.03843e-14 -0.000403 rpy=-2.95823e-30 -4.10504e-13 6.70532e-29 -> xyz=0.000136003 -9.03878e-14 -0.000403 rpy=-5.85483e-31 -1.10566e-26 -2.04919e-31
- joint revolute_3: origin xyz=0.000619747 -1.52279e-13 0.0001235 rpy=5.55112e-17 -3.87994e-13 1.94289e-16 -> xyz=0.000619747 -1.52277e-13 0.0001235 rpy=-4.61429e-16 -5.6212e-13 -1.94865e-16
- joint slider_1: parent part_1_2 -> part_1_1
- joint slider_2: origin xyz=-0.000143028 -0.00161153 0.0110102 rpy=-1.5708 3.33067e-16 -1.5708 -> xyz=-0.000143028 -0.00161153 0.0110102 rpy=-1.5708 -2.22045e-16 -1.5708; parent part_1_2 -> part_1_1

Commit message: fixes

File: models/robobee_assembly/urdf/robobee_assembly.urdf (robot description, URDF)
Before this commit: robot robobee_assembly, 32 links, 31 joints
Joints:
- joint revolute_1: limit (none) -> lower=-1.57079632679 upper=1.57079632679 effort=1 velocity=1; type continuous -> revolute
- joint revolute_1_2: limit (none) -> lower=-1.57079632679 upper=1.57079632679 effort=1 velocity=1; type continuous -> revolute

Commit message: increased transmission hinge limit
+/- 30 deg too small. now +/- 45. that is responsible for the drive "stopping" at limits.

File: models/robobee_assembly/urdf/robobee_assembly.urdf (robot description, URDF)
Before this commit: robot robobee_assembly, 32 links, 31 joints
Joints:
- joint revolute_1_3: limit lower=-0.523599 upper=0.523599 effort=1 velocity=1 -> lower=-0.7853981633974483 upper=0.7853981633974483 effort=1 velocity=1
- joint revolute_1_4: limit lower=-0.523599 upper=0.523599 effort=1 velocity=1 -> lower=-0.7853981633974483 upper=0.7853981633974483 effort=1 velocity=1
