Commit message: simulink updates
- observe that 0.01 gain is because of course you don't send 300 volts as an input signal BEFORE the amplifier
- signalsaturationlimit is some crock of shit

File: models/robobee_assembly/urdf/robobee_assembly.urdf (robot description, URDF)
Before this commit: robot robobee_assembly, 32 links, 31 joints
Links:
- link part_1_3: mass 1.70668e-06 -> 6.170668e-05

Commit message: adjusted actuator tracking

File: models/robobee_assembly/urdf/robobee_assembly.urdf (robot description, URDF)
Before this commit: robot robobee_assembly, 32 links, 31 joints
Joints:
- joint revolute_1_3: limit lower=-0.7853981633974483 upper=0.7853981633974483 effort=1 velocity=1 -> lower=-0.8727 upper=0.8727 effort=1 velocity=1
- joint revolute_1_4: limit lower=-0.7853981633974483 upper=0.7853981633974483 effort=1 velocity=1 -> lower=-0.8727 upper=0.8727 effort=1 velocity=1

Commit message: updated Ixx and URDF

File: models/robobee_assembly/urdf/robobee_assembly.urdf (robot description, URDF)
Before this commit: robot robobee_assembly, 32 links, 31 joints
Links:
- removed link part_1__1__loop_closure
- removed link part_1__2__loop_closure
- added link central_cf, mass 6.561e-06; visual mesh filename=package://robobee_assembly/meshes/Central_CF.obj scale=1 1 1
- added link central_cf_1, mass 6.561e-06; visual mesh filename=package://robobee_assembly/meshes/Central_CF.obj scale=1 1 1
- added link central_cf__1__loop_closure, mass 1e-09
- added link central_cf__1__loop_closure_1, mass 1e-09
- added link part_10, mass 1.458e-06; visual mesh filename=package://robobee_assembly/meshes/Part_10.obj scale=1 1 1
- added link part_10_1, mass 1.458e-06; visual mesh filename=package://robobee_assembly/meshes/Part_10.obj scale=1 1 1
- added link part_10__1__loop_closure, mass 1e-09
- added link part_11, mass 1.8225e-06; visual mesh filename=package://robobee_assembly/meshes/Part_11.obj scale=1 1 1
- added link part_11_1, mass 1.8225e-06; visual mesh filename=package://robobee_assembly/meshes/Part_11.obj scale=1 1 1
- added link part_12, mass 1.8225e-07; visual mesh filename=package://robobee_assembly/meshes/Part_12.obj scale=1 1 1
- added link part_12_1, mass 1.8225e-07; visual mesh filename=package://robobee_assembly/meshes/Part_12.obj scale=1 1 1
- added link part_12__1__loop_closure, mass 1e-09
- added link part_13, mass 2.27812e-07; visual mesh filename=package://robobee_assembly/meshes/Part_13.obj scale=1 1 1
- added link part_13_1, mass 2.27812e-07; visual mesh filename=package://robobee_assembly/meshes/Part_13.obj scale=1 1 1
- added link part_13__1__loop_closure, mass 1e-09
- added link part_13__1__loop_closure_1, mass 1e-09
- added link part_1__3__loop_closure, mass 1e-09
- added link part_1__4__loop_closure, mass 1e-09
- added link part_1__5__loop_closure, mass 1e-09
- added link part_4, mass 1.458e-06; visual mesh filename=package://robobee_assembly/meshes/Part_4.obj scale=1 1 1
- added link part_4_1, mass 1.458e-06; visual mesh filename=package://robobee_assembly/meshes/Part_4.obj scale=1 1 1
- added link part_5, mass 1.3365e-06; visual mesh filename=package://robobee_assembly/meshes/Part_5.obj scale=1 1 1
- added link part_5_1, mass 1.3365e-06; visual mesh filename=package://robobee_assembly/meshes/Part_5.obj scale=1 1 1
- added link part_5__1__loop_closure, mass 1e-09
- added link part_5__1__loop_closure_1, mass 1e-09
- added link part_6, mass 2.40084e-07; visual mesh filename=package://robobee_assembly/meshes/Part_6.obj scale=1 1 1
- added link part_6_1, mass 2.40084e-07; visual mesh filename=package://robobee_assembly/meshes/Part_6.obj scale=1 1 1
- added link part_6__1__loop_closure, mass 1e-09
- added link part_6__1__loop_closure_1, mass 1e-09
- added link part_7, mass 1.8225e-07; visual mesh filename=package://robobee_assembly/meshes/Part_7.obj scale=1 1 1
- added link part_7_1, mass 1.8225e-07; visual mesh filename=package://robobee_assembly/meshes/Part_7.obj scale=1 1 1
- added link part_7__1__loop_closure, mass 1e-09
- added link part_7__1__loop_closure_1, mass 1e-09
- added link part_8, mass 1.67062e-07; visual mesh filename=package://robobee_assembly/meshes/Part_8.obj scale=1 1 1
- added link part_8_1, mass 1.67062e-07; visual mesh filename=package://robobee_assembly/meshes/Part_8.obj scale=1 1 1
- added link part_8__1__loop_closure, mass 1e-09
- added link part_8__1__loop_closure_1, mass 1e-09
- added link part_9, mass 3.00105e-08; visual mesh filename=package://robobee_assembly/meshes/Part_9.obj scale=1 1 1
- added link part_9_1, mass 3.00105e-08; visual mesh filename=package://robobee_assembly/meshes/Part_9.obj scale=1 1 1
- added link part_9__1__loop_closure, mass 1e-09
- added link pzt_actuator__1_
- added link pzt_actuator__2_
- added link pzt_layer1, mass 1.38206e-05; visual mesh filename=package://robobee_assembly/meshes/PZT_Layer1.obj scale=1 1 1
- added link pzt_layer1_1, mass 1.38206e-05; visual mesh filename=package://robobee_assembly/meshes/PZT_Layer1.obj scale=1 1 1
- added link pzt_layer1__1__loop_closure, mass 1e-09
- added link pzt_layer2, mass 1.38874e-05; visual mesh filename=package://robobee_assembly/meshes/PZT_Layer2.obj scale=1 1 1
- added link pzt_layer2_1, mass 1.38874e-05; visual mesh filename=package://robobee_assembly/meshes/PZT_Layer2.obj scale=1 1 1
- added link pzt_layer2__1__loop_closure, mass 1e-09
- link part_1_2: mass 1.01477e-06 -> 1.70668e-06
- link part_1_3: mass 6.170668e-05 -> 4.38258e-06
- link part_1_4: mass 4.38258e-06 -> 1.01477e-06
Joints:
- removed joint revolute_2_loop_closure
- removed joint revolute_2_loop_closure_1
- removed joint revolute_3
- removed joint revolute_3_1
- added joint fastened_1_6: type fixed, parent transmission_right_link_base, child transmission_right_urdf__1_, origin xyz=-0.00156874 -0.000670143 -5.06127e-05 rpy=4.81906e-22 6.30258e-24 -3.87719e-26, axis -0 -0 -1
- added joint fastened_1_7: type fixed, parent wing_cf, child wing_membrane, origin xyz=-0.000247301 3.66373e-05 8e-05 rpy=4.16334e-17 -3.88578e-16 -1.92593e-33, axis 0 0 -1
- added joint fastened_5_loop_closure: type fixed, parent part_1_3, child part_1__5__loop_closure, origin xyz=-0.000934002 6.42932e-17 0.0002 rpy=-3.30869e-24 -2.14693e-15 -3.14159, axis 0 0 1
- added joint fixed_node_to_root_joint_10: type fixed, parent root, child part_11_1, origin xyz=0.000822004 3.57999e-11 0.001008 rpy=-2.53551e-15 -2.15805e-21 1.5708, axis 0 0 1
- added joint fixed_node_to_root_joint_11: type fixed, parent root, child part_10_1, origin xyz=0.000822004 3.57999e-11 0.001008 rpy=-2.53551e-15 -2.15805e-21 1.5708, axis 0 0 1
- added joint fixed_node_to_root_joint_12: type fixed, parent root, child part_13_1, origin xyz=0.000822004 3.57999e-11 0.001008 rpy=-2.53551e-15 -2.15805e-21 1.5708, axis 0 0 1
- added joint fixed_node_to_root_joint_13: type fixed, parent root, child part_5, origin xyz=-0.000822 3.57999e-11 0.001008 rpy=2.34122e-15 1.9429e-16 -1.5708, axis 0 0 1
- added joint fixed_node_to_root_joint_14: type fixed, parent root, child part_4, origin xyz=-0.000822 3.57999e-11 0.001008 rpy=2.34122e-15 1.9429e-16 -1.5708, axis 0 0 1
- added joint fixed_node_to_root_joint_15: type fixed, parent root, child pzt_layer2, origin xyz=-0.000822 3.57999e-11 0.001008 rpy=2.34122e-15 1.9429e-16 -1.5708, axis 0 0 1
- added joint fixed_node_to_root_joint_16: type fixed, parent root, child central_cf, origin xyz=-0.000822 3.57999e-11 0.001008 rpy=2.34122e-15 1.9429e-16 -1.5708, axis 0 0 1
- added joint fixed_node_to_root_joint_17: type fixed, parent root, child pzt_layer1, origin xyz=-0.000822 3.57999e-11 0.001008 rpy=2.34122e-15 1.9429e-16 -1.5708, axis 0 0 1
- added joint fixed_node_to_root_joint_18: type fixed, parent root, child part_6, origin xyz=-0.000822 3.57999e-11 0.001008 rpy=2.34122e-15 1.9429e-16 -1.5708, axis 0 0 1
- added joint fixed_node_to_root_joint_19: type fixed, parent root, child part_8, origin xyz=-0.000822 3.57999e-11 0.001008 rpy=2.34122e-15 1.9429e-16 -1.5708, axis 0 0 1
- added joint fixed_node_to_root_joint_20: type fixed, parent root, child part_12, origin xyz=-0.000822 3.57999e-11 0.001008 rpy=2.34122e-15 1.9429e-16 -1.5708, axis 0 0 1
- added joint fixed_node_to_root_joint_21: type fixed, parent root, child part_9, origin xyz=-0.000822 3.57999e-11 0.001008 rpy=2.34122e-15 1.9429e-16 -1.5708, axis 0 0 1
- added joint fixed_node_to_root_joint_22: type fixed, parent root, child part_7, origin xyz=-0.000822 3.57999e-11 0.001008 rpy=2.34122e-15 1.9429e-16 -1.5708, axis 0 0 1
- added joint fixed_node_to_root_joint_23: type fixed, parent root, child part_11, origin xyz=-0.000822 3.57999e-11 0.001008 rpy=2.34122e-15 1.9429e-16 -1.5708, axis 0 0 1
- added joint fixed_node_to_root_joint_24: type fixed, parent root, child part_10, origin xyz=-0.000822 3.57999e-11 0.001008 rpy=2.34122e-15 1.9429e-16 -1.5708, axis 0 0 1
- added joint fixed_node_to_root_joint_25: type fixed, parent root, child part_13, origin xyz=-0.000822 3.57999e-11 0.001008 rpy=2.34122e-15 1.9429e-16 -1.5708, axis 0 0 1
- added joint fixed_node_to_root_joint_26: type fixed, parent root, child part_1_4, origin xyz=-3.12792e-17 1.40187e-16 4.5e-05 rpy=-9.7945e-22 1.94289e-16 3.14159, axis 0 0 1
- added joint fixed_node_to_root_joint_27: type fixed, parent root, child part_1_3, origin xyz=2.0772e-09 -0.000775 -0.00011 rpy=9.76141e-22 -2.34122e-15 -2.22045e-16, axis 0 0 1
- added joint fixed_node_to_root_joint_28: type fixed, parent root, child part_1, origin xyz=2.0772e-09 0.000775 0.0066775 rpy=-9.7945e-22 2.34122e-15 3.14159, axis 0 0 1
- added joint fixed_node_to_root_joint_29: type fixed, parent root, child part_1_2, origin xyz=2.0772e-09 -0.0003025 0.013265 rpy=9.80322e-22 -2.34122e-15 -2.22045e-16, axis 0 0 1
- added joint fixed_node_to_root_joint_30: type fixed, parent root, child part_1_1, origin xyz=2.0772e-09 -2.75209e-08 0.00189779 rpy=2.34122e-15 1.9429e-16 -1.5708, axis 0 0 1
- added joint fixed_node_to_root_joint_31: type fixed, parent root, child transmission_base, origin xyz=-0.00421149 0.000143 0.011928 rpy=-1.5708 2.31347e-15 3.14159, axis 0 0 1
- added joint fixed_node_to_root_joint_32: type fixed, parent root, child transmission_right_link_base, origin xyz=0.00252376 -0.000639387 0.0123379 rpy=-1.5708 -2.14693e-15 -2.55351e-14, axis 0 0 1
- added joint fixed_node_to_root_joint_7: type fixed, parent root, child part_12_1, origin xyz=0.000822004 3.57999e-11 0.001008 rpy=-2.53551e-15 -2.15805e-21 1.5708, axis 0 0 1
- added joint fixed_node_to_root_joint_8: type fixed, parent root, child part_9_1, origin xyz=0.000822004 3.57999e-11 0.001008 rpy=-2.53551e-15 -2.15805e-21 1.5708, axis 0 0 1
- added joint fixed_node_to_root_joint_9: type fixed, parent root, child part_7_1, origin xyz=0.000822004 3.57999e-11 0.001008 rpy=-2.53551e-15 -2.15805e-21 1.5708, axis 0 0 1
- added joint group_1_fastened_joint_loop_closure: type fixed, parent part_4_1, child part_5__1__loop_closure, origin xyz=0 0 0 rpy=0 -0 1.50479e-44, axis -0 -0 -1
- added joint group_1_fastened_joint_loop_closure_1: type fixed, parent pzt_layer1_1, child central_cf__1__loop_closure_1, origin xyz=0 0 0 rpy=0 -0 1.50479e-44, axis 0 0 1
- added joint group_1_fastened_joint_loop_closure_10: type fixed, parent central_cf, child pzt_layer1__1__loop_closure, origin xyz=0 0 0 rpy=-3.9443e-31 -1.88079e-37 -3.15545e-30, axis -0 -0 -1
- added joint group_1_fastened_joint_loop_closure_11: type fixed, parent part_5, child part_6__1__loop_closure, origin xyz=0 0 0 rpy=-3.9443e-31 -1.88079e-37 -3.15545e-30, axis -0 -0 -1
- added joint group_1_fastened_joint_loop_closure_12: type fixed, parent part_9, child part_8__1__loop_closure_1, origin xyz=0 0 0 rpy=-3.9443e-31 -1.88079e-37 -3.15545e-30, axis 0 0 1
- added joint group_1_fastened_joint_loop_closure_13: type fixed, parent part_13, child part_12__1__loop_closure, origin xyz=0 0 0 rpy=-3.9443e-31 -1.88079e-37 -3.15545e-30, axis 0 0 1
- added joint group_1_fastened_joint_loop_closure_14: type fixed, parent part_10, child part_9__1__loop_closure, origin xyz=0 0 0 rpy=-3.9443e-31 -1.88079e-37 -3.15545e-30, axis 0 0 1
- added joint group_1_fastened_joint_loop_closure_15: type fixed, parent part_11, child part_7__1__loop_closure, origin xyz=0 0 0 rpy=-3.9443e-31 -1.88079e-37 -3.15545e-30, axis -0 -0 -1
- added joint group_1_fastened_joint_loop_closure_16: type fixed, parent part_8, child part_13__1__loop_closure, origin xyz=0 0 0 rpy=-3.9443e-31 -1.88079e-37 -3.15545e-30, axis 0 0 1
- added joint group_1_fastened_joint_loop_closure_2: type fixed, parent part_5_1, child part_6__1__loop_closure_1, origin xyz=0 0 0 rpy=0 -0 1.50479e-44, axis -0 -0 -1
- added joint group_1_fastened_joint_loop_closure_3: type fixed, parent part_9_1, child part_8__1__loop_closure, origin xyz=0 0 0 rpy=0 -0 1.50479e-44, axis 0 0 1
- added joint group_1_fastened_joint_loop_closure_4: type fixed, parent part_12_1, child part_7__1__loop_closure_1, origin xyz=0 0 0 rpy=0 -0 1.50479e-44, axis 0 0 1
- added joint group_1_fastened_joint_loop_closure_5: type fixed, parent pzt_layer2_1, child part_10__1__loop_closure, origin xyz=0 0 0 rpy=0 -0 1.50479e-44, axis 0 0 1
- added joint group_1_fastened_joint_loop_closure_6: type fixed, parent part_12_1, child part_13__1__loop_closure_1, origin xyz=0 0 0 rpy=0 -0 1.50479e-44, axis -0 -0 -1
- added joint group_1_fastened_joint_loop_closure_7: type fixed, parent part_4, child part_5__1__loop_closure_1, origin xyz=0 0 0 rpy=-3.9443e-31 -1.88079e-37 -3.15545e-30, axis -0 -0 -1
- added joint group_1_fastened_joint_loop_closure_8: type fixed, parent part_10, child pzt_layer2__1__loop_closure, origin xyz=0 0 0 rpy=-3.9443e-31 -1.88079e-37 -3.15545e-30, axis -0 -0 -1
- added joint group_1_fastened_joint_loop_closure_9: type fixed, parent pzt_layer2, child central_cf__1__loop_closure, origin xyz=0 0 0 rpy=-3.9443e-31 -1.88079e-37 -3.15545e-30, axis -0 -0 -1
- added joint revolute_2_1: type continuous, parent transmission_right_link_hinge, child transmission_right_link_2, origin xyz=0.000135962 -1.10413e-13 0.000403 rpy=-3.32479e-24 1.10071e-12 -4.33874e-30, axis -0 1 -0
- added joint revolute_2_2: type revolute, parent hinge_left_wing, child wing_cf, origin xyz=-0.00103581 -0.000520981 -7.6896e-06 rpy=4.59944e-18 -2.81431e-17 0.147079, axis -0 -0 -1, limit lower=0 upper=0 effort=1 velocity=1
- added joint revolute_3_loop_closure: type continuous, parent transmission_link_1, child transmission_link_2__1__loop_closure, origin xyz=0.000619747 -1.52277e-13 0.0001235 rpy=-4.61429e-16 -5.6212e-13 -1.94865e-16, axis -0 1 -0
- added joint revolute_3_loop_closure_1: type continuous, parent transmission_right_link_1, child transmission_right_link_2__1__loop_closure, origin xyz=0.000619747 -1.52281e-13 -0.0001235 rpy=1.17373e-16 -4.13882e-13 3.87167e-26, axis 0 -1 0
- joint fastened_1: axis 0 0 1 -> -0 1 -0; child airframe_asy__1_ -> pzt_actuator__1_; origin xyz=4.29387e-19 2.68882e-17 0.0002 rpy=4.18096e-24 1.34417e-24 6.28657e-23 -> xyz=-1.20953e-06 -0.000157 0.00384841 rpy=0 -0 1.50479e-44; parent part_1_4 -> pzt_layer1_1
- joint fastened_1_1: axis -0 -0 1 -> -0 1 -0; child wing_membrane_1 -> pzt_actuator__2_; origin xyz=-0.000989203 0.000146549 -8e-05 rpy=-1.78763e-15 -1.24258e-16 -5.27356e-16 -> xyz=-1.20953e-06 -0.000157 0.00384841 rpy=-3.9443e-31 -1.88079e-37 -3.15545e-30; parent wing_cf_1 -> pzt_layer1
- joint fastened_1_2: axis -1 -0 -0 -> 0 0 1; child hinge_left_base -> airframe_asy__1_; origin xyz=0.000531022 0.00025 -0.0001165 rpy=-3.14159 -6.93889e-17 2.55651e-17 -> xyz=4.29387e-19 2.68882e-17 0.0002 rpy=4.18096e-24 1.34417e-24 6.28657e-23; parent transmission_hinge -> part_1_3
- joint fastened_1_3: axis -0 -0 -1 -> -0 -0 1; child transmission_left_urdf__1_ -> wing_membrane_1; origin xyz=-0.0032565 -0.00108003 0.000833 rpy=-2.46517e-32 9.1608e-33 -1.12915e-64 -> xyz=-0.000989203 0.000146549 -8e-05 rpy=-1.78763e-15 -1.24258e-16 -5.27356e-16; parent transmission_base -> wing_cf_1
- joint fastened_1_4: axis -0 -0 -1 -> -1 -0 -0; child transmission_right_urdf__1_ -> hinge_left_base; origin xyz=-0.00156874 -0.000670143 -5.06127e-05 rpy=4.81906e-22 6.30258e-24 -3.87719e-26 -> xyz=0.000531022 0.00025 -0.0001165 rpy=-3.14159 -6.93889e-17 2.55651e-17; parent transmission_right_link_base -> transmission_hinge
- joint fastened_1_5: axis 0 0 -1 -> -0 -0 -1; child wing_membrane -> transmission_left_urdf__1_; origin xyz=-0.000247301 3.66373e-05 8e-05 rpy=4.16334e-17 -3.88578e-16 -1.92593e-33 -> xyz=-0.0032565 -0.00108003 0.000833 rpy=-2.46517e-32 9.1608e-33 -1.12915e-64; parent wing_cf -> transmission_base
- joint fastened_3_loop_closure: axis 0 0 1 -> -0 -0 -1; child part_1__1__loop_closure -> part_1__3__loop_closure; origin xyz=-0.000860028 8.5e-05 0.00856221 rpy=3.59382e-23 1.6075e-21 -1.5708 -> xyz=-8.5e-05 -8.5e-05 0.0037825 rpy=-1.28102e-21 3.58865e-23 1.5708; parent part_1_1 -> part_1
- joint fastened_4_loop_closure: axis 0 0 1 -> -0 -0 -1; child part_1__2__loop_closure -> part_1__4__loop_closure; origin xyz=0.00086 -0.0005575 -8.5e-05 rpy=-4.18096e-24 -1.34417e-24 -6.28657e-23 -> xyz=0.00086 -8.5e-05 0.01329 rpy=4.18096e-24 1.34417e-24 6.28657e-23
- joint fixed_node_to_root_joint: child part_1_2 -> part_5_1; origin xyz=-3.12792e-17 1.40187e-16 4.5e-05 rpy=-9.7945e-22 1.94289e-16 3.14159 -> xyz=0.000822004 3.57999e-11 0.001008 rpy=-2.53551e-15 -2.15805e-21 1.5708
- joint fixed_node_to_root_joint_1: child part_1_4 -> part_4_1; origin xyz=2.0772e-09 -0.000775 -0.00011 rpy=9.76141e-22 -2.34122e-15 -2.22045e-16 -> xyz=0.000822004 3.57999e-11 0.001008 rpy=-2.53551e-15 -2.15805e-21 1.5708
- joint fixed_node_to_root_joint_2: child part_1 -> pzt_layer2_1; origin xyz=2.0772e-09 0.000775 0.0066775 rpy=-9.7945e-22 2.34122e-15 3.14159 -> xyz=0.000822004 3.57999e-11 0.001008 rpy=-2.53551e-15 -2.15805e-21 1.5708
- joint fixed_node_to_root_joint_3: child part_1_3 -> central_cf_1; origin xyz=2.0772e-09 -0.0003025 0.013265 rpy=9.80322e-22 -2.34122e-15 -2.22045e-16 -> xyz=0.000822004 3.57999e-11 0.001008 rpy=-2.53551e-15 -2.15805e-21 1.5708
- joint fixed_node_to_root_joint_4: child part_1_1 -> pzt_layer1_1; origin xyz=2.0772e-09 -2.75209e-08 0.00189779 rpy=2.34122e-15 1.9429e-16 -1.5708 -> xyz=0.000822004 3.57999e-11 0.001008 rpy=-2.53551e-15 -2.15805e-21 1.5708
- joint fixed_node_to_root_joint_5: child transmission_base -> part_6_1; origin xyz=-0.00421149 0.000143 0.011928 rpy=-1.5708 2.31347e-15 3.14159 -> xyz=0.000822004 3.57999e-11 0.001008 rpy=-2.53551e-15 -2.15805e-21 1.5708
- joint fixed_node_to_root_joint_6: child transmission_right_link_base -> part_8_1; origin xyz=0.00252376 -0.000639387 0.0123379 rpy=-1.5708 -2.14693e-15 -2.55351e-14 -> xyz=0.000822004 3.57999e-11 0.001008 rpy=-2.53551e-15 -2.15805e-21 1.5708
- joint revolute_1: limit lower=-1.57079632679 upper=1.57079632679 effort=1 velocity=1 -> (none); type revolute -> continuous
- joint revolute_1_2: limit lower=-1.57079632679 upper=1.57079632679 effort=1 velocity=1 -> (none); type revolute -> continuous
- joint revolute_1_3: limit lower=-0.8727 upper=0.8727 effort=1 velocity=1 -> lower=-0.785398 upper=0.785398 effort=1 velocity=1
- joint revolute_1_4: limit lower=-0.8727 upper=0.8727 effort=1 velocity=1 -> lower=-0.872665 upper=0.872665 effort=1 velocity=1
- joint revolute_2: axis -0 -0 -1 -> -0 1 -0; child wing_cf -> transmission_link_2; limit lower=0 upper=0 effort=1 velocity=1 -> (none); origin xyz=-0.00103581 -0.000520981 -7.6896e-06 rpy=4.59944e-18 -2.81431e-17 0.147079 -> xyz=0.000136003 -9.03878e-14 -0.000403 rpy=-5.85483e-31 -1.10566e-26 -2.04919e-31; parent hinge_left_wing -> transmission_hinge; type revolute -> continuous

Commit message: i lwky think it works

File: models/robobee_assembly/urdf/robobee_assembly.urdf (robot description, URDF)
Before this commit: robot robobee_assembly, 78 links, 77 joints
Links:
- removed link part_10__1__loop_closure
- removed link part_13
- removed link part_13_1
- removed link part_13__1__loop_closure
- removed link part_13__1__loop_closure_1
- added link part_11__1__loop_closure, mass 1e-09
- added link part_12__1__loop_closure_1, mass 1e-09
- added link part_9__1_, mass 1e-09
- added link part_9__1__1, mass 1e-09
- added link part_9__1__loop_closure_1, mass 1e-09
- link part_1: mass 3.68516e-06 -> 3.73646e-06
- link part_10: mass 1.458e-06 -> 1.8225e-06
- link part_10_1: mass 1.458e-06 -> 1.8225e-06
- link part_11: mass 1.8225e-06 -> 1.8225e-07
- link part_11_1: mass 1.8225e-06 -> 1.8225e-07
- link part_12: mass 1.8225e-07 -> 2.27812e-07
- link part_12_1: mass 1.8225e-07 -> 2.27812e-07
- link part_1_3: mass 4.38258e-06 -> 4.43388e-06
- link part_9: mass 3.00105e-08 -> 1.458e-06
- link part_9_1: mass 3.00105e-08 -> 1.458e-06
Joints:
- joint fixed_node_to_root_joint_10: child part_11_1 -> part_10_1
- joint fixed_node_to_root_joint_11: child part_10_1 -> part_9_1
- joint fixed_node_to_root_joint_12: child part_13_1 -> part_12_1
- joint fixed_node_to_root_joint_20: child part_12 -> part_11
- joint fixed_node_to_root_joint_21: child part_9 -> part_9__1__1
- joint fixed_node_to_root_joint_23: child part_11 -> part_10
- joint fixed_node_to_root_joint_24: child part_10 -> part_9
- joint fixed_node_to_root_joint_25: child part_13 -> part_12
- joint fixed_node_to_root_joint_7: child part_12_1 -> part_11_1
- joint fixed_node_to_root_joint_8: child part_9_1 -> part_9__1_
- joint group_1_fastened_joint_loop_closure_12: parent part_9 -> part_9__1__1
- joint group_1_fastened_joint_loop_closure_13: child part_12__1__loop_closure -> part_11__1__loop_closure; parent part_13 -> part_12
- joint group_1_fastened_joint_loop_closure_14: parent part_10 -> part_9
- joint group_1_fastened_joint_loop_closure_15: parent part_11 -> part_10
- joint group_1_fastened_joint_loop_closure_16: child part_13__1__loop_closure -> part_12__1__loop_closure
- joint group_1_fastened_joint_loop_closure_3: parent part_9_1 -> part_9__1_
- joint group_1_fastened_joint_loop_closure_4: parent part_12_1 -> part_11_1
- joint group_1_fastened_joint_loop_closure_5: child part_10__1__loop_closure -> part_9__1__loop_closure_1
- joint group_1_fastened_joint_loop_closure_6: child part_13__1__loop_closure_1 -> part_12__1__loop_closure_1; parent part_12_1 -> part_11_1
- joint group_1_fastened_joint_loop_closure_8: parent part_10 -> part_9
