Commit message: restored hovering

File: models/robobee_assembly/urdf/robobee_assembly.urdf (robot description, URDF)
Before this commit: robot robobee_assembly, 78 links, 77 joints
Links:
- removed link wing_asy_right__1_
- added link wing_asy_left__1_
- link central_cf: mass 6.561e-06 -> 4.92075e-06
- link central_cf_1: mass 6.561e-06 -> 4.92075e-06
- link part_10: mass 1.8225e-06 -> 1.36688e-06
- link part_10_1: mass 1.8225e-06 -> 1.36688e-06
- link part_11: mass 1.8225e-07 -> 1.36687e-07
- link part_11_1: mass 1.8225e-07 -> 1.36687e-07
- link part_12: mass 2.27812e-07 -> 1.70859e-07
- link part_12_1: mass 2.27812e-07 -> 1.70859e-07
- link part_4: mass 1.458e-06 -> 1.0935e-06
- link part_4_1: mass 1.458e-06 -> 1.0935e-06
- link part_5: mass 1.3365e-06 -> 1.00238e-06
- link part_5_1: mass 1.3365e-06 -> 1.00238e-06
- link part_6: mass 2.40084e-07 -> 1.80063e-07
- link part_6_1: mass 2.40084e-07 -> 1.80063e-07
- link part_7: mass 1.8225e-07 -> 1.36687e-07
- link part_7_1: mass 1.8225e-07 -> 1.36687e-07
- link part_8: mass 1.67062e-07 -> 1.25297e-07
- link part_8_1: mass 1.67062e-07 -> 1.25297e-07
- link part_9: mass 1.458e-06 -> 1.0935e-06
- link part_9_1: mass 1.458e-06 -> 1.0935e-06
- link pzt_layer1: mass 1.38206e-05 -> 1.03654e-05
- link pzt_layer1_1: mass 1.38206e-05 -> 1.03654e-05
- link pzt_layer2: mass 1.38874e-05 -> 1.04156e-05
- link pzt_layer2_1: mass 1.38874e-05 -> 1.04156e-05
Joints:
- joint fastened_2_2: child wing_asy_right__1_ -> wing_asy_left__1_
